Commit message: 'Update 2110041508'

File: xela_models/urdf/allegro_hand_right.xacro (robot description, xacro)
@@ -4,4 +4,5 @@
 <xacro:include filename="$(find xela_models)/urdf/xela.xacro" />
 <link name="world" />
+<!--
 <joint name="fixed" type="fixed">
     <parent link="world" />
@@ -20,5 +21,5 @@
       </geometry>
     </collision>
-  </link>
+  </link> -->
 <!-- Notes
 Back controller covers can be disabled by setting covers to 0
@@ -26,5 +27,5 @@
 Palm sensors can be disabled by setting palm to 0
 -->
-	<xacro:allegro_hand_right sequence="1" tips="curved" parent="base_link" />
+	<xacro:allegro_hand_right sequence="1" tips="curved" parent="world" />
   <!-- Enable the following 2 if you would like to see different options the same time -->
 	<!-- <xacro:allegro_hand_right sequence="2" parent="base_link" x="0.2" tips="curved" /> -->

File: xela_models/urdf/xela.xacro (robot description, xacro)
@@ -3,8 +3,8 @@
   <!-- Rviz colors -->
   <material name="black">
-    <color rgba="0.2 0.2 0.2 1.0"/>
+    <color rgba="0.0 0.0 0.0 1.0"/>
   </material>
   <material name="blue">
-    <color rgba="0.2 0.2 0.8 1.0"/>
+    <color rgba="0.0 0.0 0.8 1.0"/>
   </material>
   <material name="green">
@@ -12,5 +12,5 @@
   </material>
   <material name="grey">
-    <color rgba="0.4 0.4 0.4 1.0"/>
+    <color rgba="0.2 0.2 0.2 1.0"/>
   </material>
   <material name="orange">
@@ -98,5 +98,5 @@
   </xacro:macro>
   <!-- Sensors -->
-  <xacro:macro name="sensoraftf" params="sequence parent x:=0.0 y:=0.0 z:=0.0 rx:=0.0 ry:=0.0 rz:=0.0 col:='blue' taxels:=0">
+  <xacro:macro name="sensoraftf" params="sequence parent x:=0.0 y:=0.0 z:=0.0 rx:=0.0 ry:=0.0 rz:=0.0 col:='blue' taxels:=0 skipinertia:=0">
     <joint name="${sequence}_aftf_fixed" type="fixed">
       <origin xyz="${x} ${y} ${z}" rpy="${radians(rx)} ${radians(ry)} ${radians(rz)}"/>
@@ -118,4 +118,12 @@
         <material name="${col}"/>
       </visual>
+      <xacro:if value="${skipinertia == 0}">
+        <inertial>
+          <mass value="0.0142" />
+          <origin xyz="0 0 0" rpy="0 0 0"/>
+          <inertia ixx="3.45e-07" ixy="0.0" ixz="0.0" iyy="3.32e-07" iyz="1.14e-08" izz="3.88e-07" />
+        </inertial>
+        <!-- will need 4x4 to be aligned without inertia (as already calculated), only for taxels -->
+      </xacro:if>
     </link>
     <link name="${sequence}_aftf_sensorbase_base_link">
@@ -163,5 +171,5 @@
     <xacro:sensor4x4 sequence="${sequence}_aftf" x="-0.0111665" y="-0.0116665" parent="${sequence}_aftf_sensorbase_base_link" body="0" taxels="${taxels}" />
   </xacro:macro>
-  <xacro:macro name="sensoraftc" params="sequence parent x:=0.0 y:=0.0 z:=0.0 rx:=0.0 ry:=0.0 rz:=0.0 col:='blue' taxels:=1">
+  <xacro:macro name="sensoraftc" params="sequence parent x:=0.0 y:=0.0 z:=0.0 rx:=0.0 ry:=0.0 rz:=0.0 col:='blue' taxels:=1 skipinertia:=0">
     <joint name="${sequence}_aftc_fixed" type="fixed">
       <origin xyz="${x-0.013} ${y} ${z}" rpy="${radians(rx)} ${radians(ry)} ${radians(rz)}"/>
@@ -183,4 +191,11 @@
         <material name="${col}"/>
       </visual>
+      <xacro:if value="${skipinertia == 0}">
+        <inertial>
+          <mass value="0.0266" />
+          <origin xyz="0 0 0" rpy="0 0 0"/>
+          <inertia ixx="1.66e-06" ixy="0.0" ixz="0.0" iyy="1.23e-06" iyz="0.0" izz="1.70e-06" />
+        </inertial>
+      </xacro:if>
     </link>
     <xacro:if value="${taxels == 1}">
@@ -217,5 +232,5 @@
     </xacro:if>
   </xacro:macro>
-   <xacro:macro name="aftd" params="sequence parent x:=0.0 y:=0.0 z:=0.0 rx:=0.0 ry:=0.0 rz:=0.0 col:='blue'">
+   <xacro:macro name="aftd" params="sequence parent x:=0.0 y:=0.0 z:=0.0 rx:=0.0 ry:=0.0 rz:=0.0 col:='blue' skipinertia:=0">
     <joint name="${sequence}_aftd_fixed" type="fixed">
       <origin xyz="${x-0.013} ${y} ${z}" rpy="${radians(rx)} ${radians(ry)} ${radians(rz)}"/>
@@ -237,7 +252,14 @@
         <material name="${col}"/>
       </visual>
+      <xacro:if value="${skipinertia == 0}">
+        <inertial>
+          <mass value="0.0168" />
+          <origin xyz="0 0 0" rpy="0 0 0"/>
+          <inertia ixx="1.63e-07" ixy="0.0" ixz="0.0" iyy="1.63e-07" iyz="0.0" izz="1.60e-07" />
+        </inertial>
+      </xacro:if>
     </link>
   </xacro:macro>
-  <xacro:macro name="sensor4x4" params="sequence parent x:=0.0 y:=0.0 z:=0.0 rx:=0.0 ry:=0.0 rz:=0.0 col:='blue' body:=1 taxels:=1">
+  <xacro:macro name="sensor4x4" params="sequence parent x:=0.0 y:=0.0 z:=0.0 rx:=0.0 ry:=0.0 rz:=0.0 col:='blue' body:=1 taxels:=1 skipinertia:=0">
     <joint name="${sequence}_4x4_fixed" type="fixed">
       <origin xyz="${x} ${y} ${z}" rpy="${radians(rx)} ${radians(ry)} ${radians(rz)}"/>
@@ -260,4 +282,11 @@
           <material name="${col}"/>
         </visual>
+        <xacro:unless value="${skipinertia == 1}">
+          <inertial>
+            <mass value="0.0036" />
+            <origin xyz="0 0 0" rpy="0 0 0"/>
+            <inertia ixx="5.76e-09" ixy="0.0" ixz="0.0" iyy="6.55e-09" iyz="1.44e-10" izz="1.20e-08" />
+          </inertial>
+        </xacro:unless>
       </xacro:if>
     </link>
@@ -281,5 +310,5 @@
     </xacro:if>
   </xacro:macro>
-  <xacro:macro name="sensor1x6" params="sequence parent x:=0.0 y:=0.0 z:=0.0 rx:=0.0 ry:=0.0 rz:=0.0 col:='blue' body:=1 taxels:=1">
+  <xacro:macro name="sensor1x6" params="sequence parent x:=0.0 y:=0.0 z:=0.0 rx:=0.0 ry:=0.0 rz:=0.0 col:='blue' body:=1 taxels:=1 skipinertia:=0">
     <joint name="${sequence}_1x6_fixed" type="fixed">
       <origin xyz="${x} ${y} ${z}" rpy="${radians(rx)} ${radians(ry)} ${radians(rz)}"/>
@@ -302,4 +331,11 @@
           <material name="${col}"/>
         </visual>
+        <xacro:unless value="${skipinertia == 1}">
+          <inertial>
+            <mass value="0.0018" />
+            <origin xyz="0 0 0" rpy="0 0 0"/>
+            <inertia ixx="9.47e-10" ixy="0.0" ixz="0.0" iyy="4.68e-11" iyz="0.0" izz="9.50e-10" />
+          </inertial>
+        </xacro:unless>
       </xacro:if>
     </link>
@@ -313,5 +349,5 @@
     </xacro:if>
   </xacro:macro>
-  <xacro:macro name="sensor4x6" params="sequence parent x:=0.0 y:=0.0 z:=0.0 rx:=0.0 ry:=0.0 rz:=0.0 col:='blue' body:=1 taxels:=1">
+  <xacro:macro name="sensor4x6" params="sequence parent x:=0.0 y:=0.0 z:=0.0 rx:=0.0 ry:=0.0 rz:=0.0 col:='blue' body:=1 taxels:=1 skipinertia:=0">
     <joint name="${sequence}_4x6_fixed" type="fixed">
       <origin xyz="${x} ${y} ${z}" rpy="${radians(rx)} ${radians(ry)} ${radians(rz)}"/>
@@ -334,4 +370,11 @@
           <material name="${col}"/>
         </visual>
+        <xacro:unless value="${skipinertia == 1}">
+          <inertial>
+            <mass value="0.0108" />
+            <origin xyz="0 0 0" rpy="0 0 0"/>
+            <inertia ixx="1.11e-07" ixy="0.0" ixz="0.0" iyy="2.97e-07" iyz="0.0" izz="4.03e-07" />
+          </inertial>
+        </xacro:unless>
       </xacro:if>
     </link>
@@ -364,6 +407,6 @@
   </xacro:macro>
   <!-- Allegro Hands -->
-  <xacro:macro name="allegro_hand_right" params="sequence parent x:=0.0 y:=0.0 z:=0.0 rx:=0.0 ry:=0.0 rz:=0.0 covers:=1 phalanges:=1 tips:='flat' palm:=1 taxels:=0">
-    <link name="${sequence}_ahr_base_link">
+  <xacro:macro name="allegro_hand_right" params="sequence parent x:=0.0 y:=0.0 z:=0.0 rx:=0.0 ry:=0.0 rz:=0.0 covers:=1 phalanges:=1 tips:='flat' palm:=1 taxels:=0 defaultnames:=0">
+    <link name="${sequence}_base_link">
       <visual>
         <geometry>
@@ -386,70 +429,143 @@
         </geometry>
       </collision>
+      <xacro:if value="${palm == 1}">
+        <inertial>
+          <mass value="0.4288" />
+          <origin xyz="0 0 0" rpy="0 0 0"/>
+          <inertia ixx="2.04e-03" ixy="8.58e-06" ixz="8.58e-06" iyy="1.23e-03" iyz="0.0" izz="1.25e-03" />
+        </inertial>
+      </xacro:if>
+      <xacro:if value="${palm != 1}">
+        <inertial>
+          <mass value="0.4154" />
+          <origin xyz="0 0 0" rpy="0 0 0"/>
+          <inertia ixx="1.87e-03" ixy="0.0" ixz="8.31e-06" iyy="1.13e-03" iyz="0.0" izz="1.11e-03" />
+        </inertial>
+      </xacro:if>
     </link>
     <joint name="${sequence}_ahr_fixed" type="fixed">
         <origin xyz="${x} ${y} ${z}" rpy="${radians(rx)} ${radians(ry)} ${radians(rz)}"/>
         <parent link="${parent}" />
-        <child link="${sequence}_ahr_base_link" />
+        <child link="${sequence}_base_link" />
       </joint>
     <xacro:if value="${palm == 1}">
-      <xacro:sensor4x6 sequence="${sequence}_ahr_palm_1" col="red" parent="${sequence}_ahr_base_link" x="0.013" y="-0.051" z="-0.0365"  rz="90" rx="90" ry="0.0" taxels="${taxels}" />
-      <xacro:sensor4x6 sequence="${sequence}_ahr_palm_2" col="green" parent="${sequence}_ahr_base_link" x="0.013" y="0.0523" z="-0.005"  rz="90" rx="90" ry="180.0" taxels="${taxels}" />
-      <xacro:sensor4x6 sequence="${sequence}_ahr_palm_3" col="blue" parent="${sequence}_ahr_base_link" x="0.013" y="-0.051" z="-0.068" rz="90" rx="90" ry="0.0" taxels="${taxels}" />
-    </xacro:if>
+      <xacro:sensor4x6 sequence="${sequence}_ahr_palm_1" col="red" parent="${sequence}_base_link" x="0.013" y="-0.051" z="-0.0365"  rz="90" rx="90" ry="0.0" taxels="${taxels}" skipinertia="1" />
+      <xacro:sensor4x6 sequence="${sequence}_ahr_palm_2" col="green" parent="${sequence}_base_link" x="0.013" y="0.0523" z="-0.005"  rz="90" rx="90" ry="180.0" taxels="${taxels}" skipinertia="1" />
+      <xacro:sensor4x6 sequence="${sequence}_ahr_palm_3" col="blue" parent="${sequence}_base_link" x="0.013" y="-0.051" z="-0.068" rz="90" rx="90" ry="0.0" taxels="${taxels}" skipinertia="1" />
+    </xacro:if>
+    <xacro:if value="${defaultnames == 1}">
     <xacro:finger
-      sequence=			"${sequence}_hitosashi_finger"
-      parent=				"${sequence}_ahr_base_link"
-      finger_num=			"0"
+      sequence=			    "${sequence}"
+      parent=				    "${sequence}_base_link"
+      finger_num=			  "0"
       offset_origin_x=	"${0}"
       offset_origin_y=	"${0.0435}"
       offset_origin_z=	"${-0.001542}"
       finger_angle_r=		"-${radians(5.0)}"
-      covers=				"${covers}"
+      covers=				    "${covers}"
       phalanges=				"${phalanges}"
-      tip=				"${tips}"
-      taxels=     "${taxels}"
+      tip=				      "${tips}"
+      taxels=           "${taxels}"
     />
     <xacro:finger
-      sequence=			"${sequence}_naka_finger"
-      parent=				"${sequence}_ahr_base_link"
-      finger_num=			"1"
+      sequence=			    "${sequence}"
+      parent=				    "${sequence}_base_link"
+      finger_num=			  "1"
       offset_origin_x=	"${0}"
       offset_origin_y=	"0"
       offset_origin_z=	"${0.0007}"
       finger_angle_r=		"0.0"
-      covers=				"${covers}"
+      covers=				    "${covers}"
       phalanges=				"${phalanges}"
-      tip=				"${tips}"
-      taxels=     "${taxels}"
+      tip=				      "${tips}"
+      taxels=           "${taxels}"
     />
     <xacro:finger
-      sequence=			"${sequence}_kusuri_finger"
-      parent=				"${sequence}_ahr_base_link"
-      finger_num=			"2"
+      sequence=			    "${sequence}"
+      parent=				    "${sequence}_base_link"
+      finger_num=			  "2"
       offset_origin_x=	"${0}"
       offset_origin_y=	"-${0.0435}"
       offset_origin_z=	"${-0.001542}"
       finger_angle_r=		"${radians(5.0)}"
-      covers=				"${covers}"
+      covers=				    "${covers}"
       phalanges=				"${phalanges}"
-      tip=				"${tips}"
-      taxels=     "${taxels}"
+      tip=				      "${tips}"
+      taxels=           "${taxels}"
     />
     <xacro:thumb_right
-      sequence=			"${sequence}_oya_finger"
-      parent=				"${sequence}_ahr_base_link"
-      finger_num=			"3"
+      sequence=			    "${sequence}"
+      parent=				    "${sequence}_base_link"
+      finger_num=			  "3"
       offset_origin_x=	"-0.0182"
       offset_origin_y=	"0.019333"
       offset_origin_z=	"-0.045987"
-      covers=				"${covers}"
+      covers=				    "${covers}"
       finger_angle_r=		"0"
       finger_angle_p=		"-${radians(95)}"
       finger_angle_y=		"-${radians(90)}"
       phalanges=				"${phalanges}"
-      tip=				"${tips}"
-      taxels=     "${taxels}"
+      tip=				      "${tips}"
+      taxels=           "${taxels}"
     />
+    </xacro:if>
+    <xacro:unless value="${defaultnames == 1}">
+      <xacro:finger
+        sequence=			    "${sequence}_hitosashi_finger"
+        parent=				    "${sequence}_base_link"
+        finger_num=			  "0"
+        offset_origin_x=	"${0}"
+        offset_origin_y=	"${0.0435}"
+        offset_origin_z=	"${-0.001542}"
+        finger_angle_r=		"-${radians(5.0)}"
+        covers=				    "${covers}"
+        phalanges=				"${phalanges}"
+        tip=				      "${tips}"
+        taxels=           "${taxels}"
+      />
+      <xacro:finger
+        sequence=			    "${sequence}_naka_finger"
+        parent=				    "${sequence}_base_link"
+        finger_num=			  "1"
+        offset_origin_x=	"${0}"
+        offset_origin_y=	"0"
+        offset_origin_z=	"${0.0007}"
+        finger_angle_r=		"0.0"
+        covers=				    "${covers}"
+        phalanges=				"${phalanges}"
+        tip=				      "${tips}"
+        taxels=           "${taxels}"
+      />
+      <xacro:finger
+        sequence=			    "${sequence}_kusuri_finger"
+        parent=				    "${sequence}_base_link"
+        finger_num=			  "2"
+        offset_origin_x=	"${0}"
+        offset_origin_y=	"-${0.0435}"
+        offset_origin_z=	"${-0.001542}"
+        finger_angle_r=		"${radians(5.0)}"
+        covers=				    "${covers}"
+        phalanges=				"${phalanges}"
+        tip=				      "${tips}"
+        taxels=           "${taxels}"
+      />
+      <xacro:thumb_right
+        sequence=			    "${sequence}_oya_finger"
+        parent=				    "${sequence}_base_link"
+        finger_num=			  "3"
+        offset_origin_x=	"-0.0182"
+        offset_origin_y=	"0.019333"
+        offset_origin_z=	"-0.045987"
+        covers=				    "${covers}"
+        finger_angle_r=		"0"
+        finger_angle_p=		"-${radians(95)}"
+        finger_angle_y=		"-${radians(90)}"
+        phalanges=				"${phalanges}"
+        tip=				      "${tips}"
+        taxels=           "${taxels}"
+      />
+    </xacro:unless>
     </xacro:macro>
+    <!--FINGER MACRO-->
     <xacro:macro name="finger" params="sequence parent finger_num offset_origin_x offset_origin_y offset_origin_z finger_angle_r covers:=1 tip:='flat' phalanges:=1 taxels:=0">
       <link name="${sequence}_finger_link_${finger_num*4+0}">
@@ -466,4 +582,9 @@
           <origin rpy="0 0 0" xyz="0 0 ${0.0164/2+0.003}"/>
         </collision>
+        <inertial>
+          <mass value="0.0127" />
+          <origin xyz="0 0 0" rpy="0 0 0"/>
+          <inertia ixx="1.38e-07" ixy="1.27e-10" ixz="4.83e-09" iyy="6.83e-08" iyz="0.0" izz="1.16e-07" />
+        </inertial>
       </link>
       <joint name="${sequence}_finger_joint_${finger_num*4+0}" type="revolute">
@@ -492,6 +613,29 @@
           <origin rpy="0 0 0" xyz="0 0 ${0.0164/2}"/>
         </collision>
+        <xacro:if value="${covers == 1}">
+          <inertial>
+            <mass value="0.0809" />
+            <origin xyz="0 0 0" rpy="0 0 0"/>
+            <inertia ixx="1.75e-05" ixy="0.0" ixz="5.66e-08" iyy="1.80e-05" iyz="0.0" izz="4.60e-06" />
+          </inertial>
+        </xacro:if>
+        <xacro:unless value="${covers == 1}">
+          <xacro:if value="${phalanges == 1}">
+            <inertial>
+              <mass value="0.0719" />
+              <origin xyz="0 0 0" rpy="0 0 0"/>
+              <inertia ixx="1.56e-05" ixy="0.0" ixz="5.03e-08" iyy="1.60e-05" iyz="0.0" izz="4.09e-06" />
+            </inertial>
+          </xacro:if>
+          <xacro:unless value="${phalanges == 1}">
+            <inertial>
+              <mass value="0.0650" />
+              <origin xyz="0 0 0" rpy="0 0 0"/>
+              <inertia ixx="1.14e-05" ixy="0.0" ixz="0.0" iyy="1.12e-05" iyz="0.0" izz="2.56e-06" />
+            </inertial>
+          </xacro:unless>
+        </xacro:unless>
       </link>
-      <xacro:if value="${covers == 1}">
+      <xacro:if value="${covers == 1}"><!--covers are always with sensors-->
         <link name="${sequence}_finger_link_${finger_num*4+1}_cover">
           <visual>
@@ -507,4 +651,5 @@
             <origin rpy="0 0 0" xyz="0 0 ${0.0177/2}"/>
           </collision>
+          <!--As link is fixed, inertias will be inside the main link-->
         </link>
         <joint name="${sequence}_finger_link_${finger_num*4+1}_cover_joint" type="fixed">
@@ -515,6 +660,6 @@
       </xacro:if>
       <xacro:if value="${phalanges == 1}">
-        <xacro:sensor4x4 sequence="${sequence}_finger_link_${finger_num*4+1}A" col="red" parent="${sequence}_finger_link_${finger_num*4+1}" ry="-90" rz="180" z="0.033" y="0.012" x="0.0108" body="0" taxels="${taxels}" />
-        <xacro:sensor4x4 sequence="${sequence}_finger_link_${finger_num*4+1}B" col="red" parent="${sequence}_finger_link_${finger_num*4+1}" ry="90" z="0.021" y="-0.012" x="0.0108" body="0" taxels="${taxels}" />
+        <xacro:sensor4x4 sequence="${sequence}_finger_link_${finger_num*4+1}A" col="red" parent="${sequence}_finger_link_${finger_num*4+1}" ry="-90" rz="180" z="0.033" y="0.012" x="0.0108" body="0" taxels="${taxels}" skipinertia="1" />
+        <xacro:sensor4x4 sequence="${sequence}_finger_link_${finger_num*4+1}B" col="red" parent="${sequence}_finger_link_${finger_num*4+1}" ry="90" z="0.021" y="-0.012" x="0.0108" body="0" taxels="${taxels}" skipinertia="1" />
       </xacro:if>
       <joint name="${sequence}_finger_joint_${finger_num*4+1}" type="revolute">
@@ -523,5 +668,5 @@
         <parent link="${sequence}_finger_link_${finger_num*4+0}"/>
         <child link="${sequence}_finger_link_${finger_num*4+1}"/>
-        <origin xyz="0 0 ${0.0164+0.004}"/> <!-- New height on fingers -->
+        <origin xyz="0 0 ${0.0164+0.004}"/><!-- New height on fingers -->
       </joint>
       <link name="${sequence}_finger_link_${finger_num*4+2}">
@@ -543,4 +688,27 @@
           <origin rpy="0 0 0" xyz="0 0 ${0.0540/2}"/>
         </collision>
+        <xacro:if value="${covers == 1}"><!--covers are always with sensors-->
+          <inertial>
+            <mass value="0.0447" />
+            <origin xyz="0 0 0" rpy="0 0 0"/>
+            <inertia ixx="3.80e-07" ixy="0.0" ixz="7.15e-09" iyy="2.26e-07" iyz="1.34e-09" izz="1.86e-07" />
+          </inertial>
+        </xacro:if>
+        <xacro:unless value="${covers == 1}">
+          <xacro:if value="${phalanges == 1}">
+            <inertial>
+              <mass value="0.0422" />
+              <origin xyz="0 0 0" rpy="0 0 0"/>
+              <inertia ixx="3.15e-06" ixy="0.0" ixz="0.0" iyy="3.05e-06" iyz="0.0" izz="1.33e-06" />
+            </inertial>
+          </xacro:if>
+          <xacro:unless value="${phalanges == 1}">
+            <inertial>
+              <mass value="0.0355" />
+              <origin xyz="0 0 0" rpy="0 0 0"/>
+              <inertia ixx="2.46e-06" ixy="0.0" ixz="0.0" iyy="2.26e-06" iyz="0.0" izz="8.95e-07" />
+            </inertial>
+          </xacro:unless>
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