Commit message: 'Update 2110121045'

File: xela_models/urdf/allegro_hand_right.xacro (robot description, xacro)
@@ -9,5 +9,5 @@
 Palm sensors can be disabled by setting palm to 0
 -->
-	<xacro:allegro_hand_right sequence="" tips="curved" parent="world" />
+	<xacro:allegro_hand_right sequence="" tips="curved" parent="world" defaultnames="1" />
   <!-- Enable the following 2 if you would like to see different options the same time -->
 	<!-- <xacro:allegro_hand_right sequence="2" parent="world" x="0.2" tips="curved" /> -->

File: xela_models/urdf/xela.xacro (robot description, xacro)
@@ -108,5 +108,5 @@
         <origin xyz="0 0 0" rpy="0 0 0" />
         <geometry>
-          <mesh filename="package://xela_models/mesh/ft_f_collision.stl"/>
+          <mesh filename="package://xela_models/mesh/ft_f.stl"/>
         </geometry>
       </collision>
@@ -114,5 +114,5 @@
         <origin xyz="0 0 0" rpy="0 0 0" />
         <geometry>
-          <mesh filename="package://xela_models/mesh/ft_f_visual.stl"/>
+          <mesh filename="package://xela_models/mesh/ft_f.stl"/>
         </geometry>
         <material name="${col}"/>
@@ -124,5 +124,4 @@
           <inertia ixx="3.45e-07" ixy="0.0" ixz="0.0" iyy="3.32e-07" iyz="1.14e-08" izz="3.88e-07" />
         </inertial>
-        <!-- will need 4x4 to be aligned without inertia (as already calculated), only for taxels -->
       </xacro:if>
     </link>
@@ -169,5 +168,7 @@
       <limit effort="100.0" lower="0.000" upper="0.000" velocity="0.5"/>
     </joint>
-    <xacro:sensor4x4 sequence="${sequence}_aftf" x="-0.0111665" y="-0.0116665" parent="${sequence}_aftf_sensorbase_base_link" body="0" taxels="${taxels}" />
+    <xacro:if value="${taxels==1}">
+      <xacro:sensor4x4 sequence="${sequence}_aftf" x="-0.0111665" y="-0.0116665" parent="${sequence}_aftf_sensorbase_base_link" body="0" />
+    </xacro:if>
   </xacro:macro>
   <xacro:macro name="sensoraftc" params="sequence parent x:=0.0 y:=0.0 z:=0.0 rx:=0.0 ry:=0.0 rz:=0.0 col:='blue' taxels:=1 skipinertia:=0">
@@ -181,5 +182,5 @@
         <origin xyz="0 0 0" rpy="0 0 0" />
         <geometry>
-          <mesh filename="package://xela_models/mesh/ft_c_collision.stl"/>
+          <mesh filename="package://xela_models/mesh/ft_c.stl"/>
         </geometry>
       </collision>
@@ -187,5 +188,5 @@
         <origin xyz="0 0 0" rpy="0 0 0" />
         <geometry>
-          <mesh filename="package://xela_models/mesh/ft_c_visual.stl"/>
+          <mesh filename="package://xela_models/mesh/ft_c.stl"/>
         </geometry>
         <material name="${col}"/>
@@ -518,5 +519,5 @@
     <xacro:unless value="${defaultnames == 1}">
       <xacro:finger
-        sequence=			    "${seq}hitosashi_finger"
+        sequence=			    "${seq}hitosashi_finger_"
         parent=				    "${seq}base_link"
         finger_num=			  "0"
@@ -531,5 +532,5 @@
       />
       <xacro:finger
-        sequence=			    "${seq}naka_finger"
+        sequence=			    "${seq}naka_finger_"
         parent=				    "${seq}base_link"
         finger_num=			  "1"
@@ -544,5 +545,5 @@
       />
       <xacro:finger
-        sequence=			    "${seq}kusuri_finger"
+        sequence=			    "${seq}kusuri_finger_"
         parent=				    "${seq}base_link"
         finger_num=			  "2"
@@ -557,5 +558,5 @@
       />
       <xacro:thumb_right
-        sequence=			    "${seq}oya_finger"
+        sequence=			    "${seq}oya_finger_"
         parent=				    "${seq}base_link"
         finger_num=			  "3"
@@ -575,5 +576,5 @@
     <!--FINGER MACRO-->
     <xacro:macro name="finger" params="sequence parent finger_num offset_origin_x offset_origin_y offset_origin_z finger_angle_r covers:=1 tip:='flat' phalanges:=1 taxels:=0">
-      <link name="${sequence}_finger_link_${finger_num*4+0}">
+      <link name="${sequence}finger_link_${finger_num*4+0}">
         <visual>
           <geometry>
@@ -594,12 +595,12 @@
         </inertial>
       </link>
-      <joint name="${sequence}_finger_joint_${finger_num*4+0}" type="revolute">
+      <joint name="${sequence}finger_joint_${finger_num*4+0}" type="revolute">
         <axis xyz="0 0 1"/>
         <limit effort="15" velocity="7" lower="${-0.57+0.1}" upper="${0.57-0.1}" />
         <parent link="${parent}"/>
-        <child link="${sequence}_finger_link_${finger_num*4+0}"/>
+        <child link="${sequence}finger_link_${finger_num*4+0}"/>
         <origin rpy="${finger_angle_r} 0 0" xyz="${offset_origin_x} ${offset_origin_y} ${offset_origin_z}"/>
       </joint>
-      <link name="${sequence}_finger_link_${finger_num*4+1}">
+      <link name="${sequence}finger_link_${finger_num*4+1}">
         <visual>
           <geometry>
@@ -644,5 +645,5 @@
       </link>
       <xacro:if value="${covers == 1}"><!--covers are always with sensors-->
-        <link name="${sequence}_finger_link_${finger_num*4+1}_cover">
+        <link name="${sequence}finger_link_${finger_num*4+1}_cover">
           <visual>
             <geometry>
@@ -659,22 +660,22 @@
           <!--As link is fixed, inertias will be inside the main link-->
         </link>
-        <joint name="${sequence}_finger_link_${finger_num*4+1}_cover_joint" type="fixed">
+        <joint name="${sequence}finger_link_${finger_num*4+1}_cover_joint" type="fixed">
           <origin xyz="0.0 0.0 0.0" rpy="0.0 0.0 0.0"/>
-          <parent link="${sequence}_finger_link_${finger_num*4+1}" />
-          <child link="${sequence}_finger_link_${finger_num*4+1}_cover" />
+          <parent link="${sequence}finger_link_${finger_num*4+1}" />
+          <child link="${sequence}finger_link_${finger_num*4+1}_cover" />
         </joint>
       </xacro:if>
-      <xacro:if value="${phalanges == 1}">
-        <xacro:sensor4x4 sequence="${sequence}_finger_link_${finger_num*4+1}A" col="red" parent="${sequence}_finger_link_${finger_num*4+1}" ry="-90" rz="180" z="0.033" y="0.012" x="0.0108" body="0" taxels="${taxels}" skipinertia="1" />
-        <xacro:sensor4x4 sequence="${sequence}_finger_link_${finger_num*4+1}B" col="red" parent="${sequence}_finger_link_${finger_num*4+1}" ry="90" z="0.021" y="-0.012" x="0.0108" body="0" taxels="${taxels}" skipinertia="1" />
-      </xacro:if>
-      <joint name="${sequence}_finger_joint_${finger_num*4+1}" type="revolute">
+      <xacro:if value="${phalanges == 1 and taxels == 1}">
+        <xacro:sensor4x4 sequence="${sequence}finger_link_${finger_num*4+1}A" col="red" parent="${sequence}finger_link_${finger_num*4+1}" ry="-90" rz="180" z="0.033" y="0.012" x="0.0108" body="0" taxels="${taxels}" skipinertia="1" />
+        <xacro:sensor4x4 sequence="${sequence}finger_link_${finger_num*4+1}B" col="red" parent="${sequence}finger_link_${finger_num*4+1}" ry="90" z="0.021" y="-0.012" x="0.0108" body="0" taxels="${taxels}" skipinertia="1" />
+      </xacro:if>
+      <joint name="${sequence}finger_joint_${finger_num*4+1}" type="revolute">
         <limit effort="15" velocity="7" lower="${-0.296+0.1}" upper="${1.71-0.1}" />
         <axis xyz="0 1 0"/>
-        <parent link="${sequence}_finger_link_${finger_num*4+0}"/>
-        <child link="${sequence}_finger_link_${finger_num*4+1}"/>
+        <parent link="${sequence}finger_link_${finger_num*4+0}"/>
+        <child link="${sequence}finger_link_${finger_num*4+1}"/>
         <origin xyz="0 0 ${0.0164+0.004}"/><!-- New height on fingers -->
       </joint>
-      <link name="${sequence}_finger_link_${finger_num*4+2}">
+      <link name="${sequence}finger_link_${finger_num*4+2}">
         <visual>
           <geometry>
@@ -719,5 +720,5 @@
       </link>
       <xacro:if value="${covers == 1}">
-        <link name="${sequence}_finger_link_${finger_num*4+2}_cover">
+        <link name="${sequence}finger_link_${finger_num*4+2}_cover">
           <visual>
             <geometry>
@@ -733,21 +734,21 @@
           </collision>
         </link>
-        <joint name="${sequence}_finger_link_${finger_num*4+2}_cover_joint" type="fixed">
+        <joint name="${sequence}finger_link_${finger_num*4+2}_cover_joint" type="fixed">
           <origin xyz="0.0 0.0 0.0" rpy="0.0 0.0 0.0"/>
-          <parent link="${sequence}_finger_link_${finger_num*4+2}" />
-          <child link="${sequence}_finger_link_${finger_num*4+2}_cover" />
+          <parent link="${sequence}finger_link_${finger_num*4+2}" />
+          <child link="${sequence}finger_link_${finger_num*4+2}_cover" />
         </joint>
       </xacro:if>
-      <xacro:if value="${phalanges == 1}">
-        <xacro:sensor4x4 sequence="${sequence}_finger_link_${finger_num*4+2}" col="red" parent="${sequence}_finger_link_${finger_num*4+2}" ry="90" z="0.0445" y="-0.012" x="0.01" body="0" taxels="${taxels}" skipinertia="1" />
-      </xacro:if>
-      <joint name="${sequence}_finger_joint_${finger_num*4+2}" type="revolute">
+      <xacro:if value="${phalanges == 1 and taxels == 1}">
+        <xacro:sensor4x4 sequence="${sequence}finger_link_${finger_num*4+2}" col="red" parent="${sequence}finger_link_${finger_num*4+2}" ry="90" z="0.0445" y="-0.012" x="0.01" body="0" skipinertia="1" />
+      </xacro:if>
+      <joint name="${sequence}finger_joint_${finger_num*4+2}" type="revolute">
         <axis xyz="0 1 0"/>
         <limit effort="15" velocity="7" lower="${-0.274+0.1}" upper="${1.809-0.1}" />
-        <parent link="${sequence}_finger_link_${finger_num*4+1}"/>
-        <child link="${sequence}_finger_link_${finger_num*4+2}"/>
+        <parent link="${sequence}finger_link_${finger_num*4+1}"/>
+        <child link="${sequence}finger_link_${finger_num*4+2}"/>
         <origin xyz="0 0 ${0.0540}"/>
       </joint>
-      <link name="${sequence}_finger_link_${finger_num*4+3}">
+      <link name="${sequence}finger_link_${finger_num*4+3}">
         <visual>
           <geometry>
@@ -784,19 +785,19 @@
         </xacro:unless>
       </link>
-      <joint name="${sequence}_finger_joint_${finger_num*4+3}" type="revolute">
+      <joint name="${sequence}finger_joint_${finger_num*4+3}" type="revolute">
         <axis xyz="0 1 0"/>
         <limit effort="15" velocity="7" lower="${-0.327+0.1}" upper="${1.718-0.1}" />
-        <parent link="${sequence}_finger_link_${finger_num*4+2}"/>
-        <child link="${sequence}_finger_link_${finger_num*4+3}"/>
+        <parent link="${sequence}finger_link_${finger_num*4+2}"/>
+        <child link="${sequence}finger_link_${finger_num*4+3}"/>
         <origin xyz="0 0.0 0.0384"/>
       </joint>
     <xacro:if value="${tip == 'flat'}">
-      <xacro:sensoraftf sequence="${sequence}_finger_${finger_num}" col="red" parent="${sequence}_finger_link_${finger_num*4+3}" rx="90" rz="90" z="0.016" taxels="${taxels}" skipinertia="1"/>
+      <xacro:sensoraftf sequence="${sequence}finger_${finger_num}" col="red" parent="${sequence}finger_link_${finger_num*4+3}" rx="90" rz="90" z="0.016" taxels="${taxels}" skipinertia="1"/>
     </xacro:if>
     <xacro:if value="${tip == 'curved'}">
-      <xacro:sensoraftc sequence="${sequence}_finger_${finger_num}" col="red" parent="${sequence}_finger_link_${finger_num*4+3}" rx="90" rz="90" z="0.016" taxels="${taxels}" skipinertia="1"/>
+      <xacro:sensoraftc sequence="${sequence}finger_${finger_num}" col="red" parent="${sequence}finger_link_${finger_num*4+3}" rx="90" rz="90" z="0.016" taxels="${taxels}" skipinertia="1"/>
     </xacro:if>
     <xacro:if value="${tip == 'default'}">
-      <xacro:aftd sequence="${sequence}_finger_${finger_num}" col="white" parent="${sequence}_finger_link_${finger_num*4+3}" rx="0" rz="0" z="0.027" x="0.013" skipinertia="1"/>
+      <xacro:aftd sequence="${sequence}finger_${finger_num}" col="white" parent="${sequence}finger_link_${finger_num*4+3}" rx="0" rz="0" z="0.027" x="0.013" skipinertia="1"/>
     </xacro:if>
     </xacro:macro>
@@ -939,6 +940,6 @@
         </joint>
       </xacro:if>
-      <xacro:if value="${phalanges == 1}">
-        <xacro:sensor4x4 sequence="${sequence}_link_${finger_num*4+2}" parent="${sequence}_link_${finger_num*4+2}" ry="90" z="0.023" y="-0.012" x="0.011" body="0" taxels="${taxels}" skipinertia="1" />
+      <xacro:if value="${phalanges == 1 and taxels == 1}">
+        <xacro:sensor4x4 sequence="${sequence}_link_${finger_num*4+2}" parent="${sequence}_link_${finger_num*4+2}" ry="90" z="0.023" y="-0.012" x="0.011" body="0" skipinertia="1" />
       </xacro:if>
       <joint name="${sequence}_joint_${finger_num*4+2}" type="revolute">
@@ -1039,6 +1040,6 @@
         </xacro:unless>
       </link>
-      <xacro:if value="${phalanges == 1}">
-        <xacro:sensor4x4 sequence="${sequence}_link_${finger_num*4+3}" parent="${sequence}_link_${finger_num*4+3}" ry="90" z="0.021" y="-0.012" x="0.011" body="0" taxels="${taxels}" skipinertia="1" />
+      <xacro:if value="${phalanges == 1 and taxels == 1}">
+        <xacro:sensor4x4 sequence="${sequence}_link_${finger_num*4+3}" parent="${sequence}_link_${finger_num*4+3}" ry="90" z="0.021" y="-0.012" x="0.011" body="0" skipinertia="1" />
       </xacro:if>
     <joint name="${sequence}_joint_${finger_num*4+3}" type="revolute">
