Commit message: 1.2.5-dev-210+380852

File: xela_models/urdf/xela.xacro (robot description, xacro)
@@ -118,4 +118,9 @@
         <material name="${col}"/>
       </visual>
+      <inertial><!-- TO FILL IN-->
+        <origin xyz="0.0 0.0 0.0" rpy="0.0 0.0 0.0"/>
+        <mass value="0.0"/>
+        <inertia ixx="0.0" ixy="0.0" ixz="0.0" iyy="0.0" iyz="0.0" izz="0.0"/>
+      </inertial>
     </link>
     <link name="${sequence}_aftf_sensorbase_base_link">
@@ -125,5 +130,5 @@
         </geometry>
         <origin xyz="0.0 0.0 0.0" rpy="0 0 0"/>
-        <material name="black"/>
+        <material name="black" />
       </visual>
       <collision>
@@ -139,5 +144,5 @@
         </geometry>
         <origin xyz="0.0 0.0 0.0" rpy="0 0 0"/>
-        <material name="black"/>
+        <material name="black" />
       </visual>
       <collision>
@@ -183,4 +188,9 @@
         <material name="${col}"/>
       </visual>
+      <inertial><!-- TO FILL IN-->
+        <origin xyz="0.0 0.0 0.0" rpy="0.0 0.0 0.0"/>
+        <mass value="0.0"/>
+        <inertia ixx="0.0" ixy="0.0" ixz="0.0" iyy="0.0" iyz="0.0" izz="0.0"/>
+      </inertial>
     </link>
     <xacro:if value="${taxels == 1}">
@@ -237,4 +247,9 @@
         <material name="${col}"/>
       </visual>
+      <inertial><!-- TO FILL IN (Allegro defaults)-->
+        <origin xyz="0.0 0.0 0.0" rpy="0.0 0.0 0.0"/>
+        <mass value="0.0"/>
+        <inertia ixx="0.0" ixy="0.0" ixz="0.0" iyy="0.0" iyz="0.0" izz="0.0"/>
+      </inertial>
     </link>
   </xacro:macro>
@@ -261,4 +276,9 @@
         </visual>
       </xacro:if>
+      <inertial><!-- TO FILL IN-->
+        <origin xyz="0.0 0.0 0.0" rpy="0.0 0.0 0.0"/>
+        <mass value="0.0"/>
+        <inertia ixx="0.0" ixy="0.0" ixz="0.0" iyy="0.0" iyz="0.0" izz="0.0"/>
+      </inertial>
     </link>
     <xacro:if value="${taxels == 1}">
@@ -303,4 +323,9 @@
         </visual>
       </xacro:if>
+      <inertial><!-- TO FILL IN-->
+        <origin xyz="0.0 0.0 0.0" rpy="0.0 0.0 0.0"/>
+        <mass value="0.0"/>
+        <inertia ixx="0.0" ixy="0.0" ixz="0.0" iyy="0.0" iyz="0.0" izz="0.0"/>
+      </inertial>
     </link>
     <xacro:if value="${taxels == 1}">
@@ -335,4 +360,9 @@
         </visual>
       </xacro:if>
+      <inertial><!-- TO FILL IN-->
+        <origin xyz="0.0 0.0 0.0" rpy="0.0 0.0 0.0"/>
+        <mass value="0.0"/>
+        <inertia ixx="0.0" ixy="0.0" ixz="0.0" iyy="0.0" iyz="0.0" izz="0.0"/>
+      </inertial>
     </link>
     <xacro:if value="${taxels == 1}">
@@ -386,4 +416,9 @@
         </geometry>
       </collision>
+      <inertial><!-- TO FILL IN BASE-->
+        <origin xyz="0.0 0.0 0.0" rpy="0.0 0.0 0.0"/>
+        <mass value="0.0"/>
+        <inertia ixx="0.0" ixy="0.0" ixz="0.0" iyy="0.0" iyz="0.0" izz="0.0"/>
+      </inertial>
     </link>
     <joint name="${sequence}_ahr_fixed" type="fixed">
@@ -466,8 +501,13 @@
           <origin rpy="0 0 0" xyz="0 0 ${0.0164/2+0.003}"/>
         </collision>
+        <inertial><!-- TO FILL IN-->
+          <origin xyz="0.0 0.0 0.0" rpy="0.0 0.0 0.0"/>
+          <mass value="0.0"/>
+          <inertia ixx="0.0" ixy="0.0" ixz="0.0" iyy="0.0" iyz="0.0" izz="0.0"/>
+        </inertial>
       </link>
       <joint name="${sequence}_finger_joint_${finger_num*4+0}" type="revolute">
         <axis xyz="0 0 1"/>
-        <limit effort="0" velocity="0" lower="${-0.57+0.1}" upper="${0.57-0.1}" />
+        <limit effort="15" velocity="7" lower="${-0.57+0.1}" upper="${0.57-0.1}" />
         <parent link="${parent}"/>
         <child link="${sequence}_finger_link_${finger_num*4+0}"/>
@@ -484,12 +524,17 @@
             </xacro:if>
           </geometry>
-          <material name="black"/>
+          <material name="black" />
         </visual>
         <collision>
           <geometry>
-            <box size="${0.0196} ${0.0275} ${0.0540}"/>
-          </geometry>
-          <origin rpy="0 0 0" xyz="0 0 ${0.0540/2}"/>
+            <box size="${0.0196} ${0.0275} ${0.0164}"/>
+          </geometry>
+          <origin rpy="0 0 0" xyz="0 0 ${0.0164/2}"/>
         </collision>
+        <inertial><!-- TO FILL IN-->
+          <origin xyz="0.0 0.0 0.0" rpy="0.0 0.0 0.0"/>
+          <mass value="0.0"/>
+          <inertia ixx="0.0" ixy="0.0" ixz="0.0" iyy="0.0" iyz="0.0" izz="0.0"/>
+        </inertial>
       </link>
       <xacro:if value="${covers == 1}">
@@ -507,9 +552,14 @@
             <origin rpy="0 0 0" xyz="0 0 ${0.0177/2}"/>
           </collision>
+          <inertial><!-- TO FILL IN-->
+            <origin xyz="0.0 0.0 0.0" rpy="0.0 0.0 0.0"/>
+            <mass value="0.0"/>
+            <inertia ixx="0.0" ixy="0.0" ixz="0.0" iyy="0.0" iyz="0.0" izz="0.0"/>
+          </inertial>
         </link>
         <joint name="${sequence}_finger_link_${finger_num*4+1}_cover_joint" type="fixed">
-        <origin xyz="0.0 0.0 0.0" rpy="0.0 0.0 0.0"/>
-        <parent link="${sequence}_finger_link_${finger_num*4+1}" />
-        <child link="${sequence}_finger_link_${finger_num*4+1}_cover" />
+          <origin xyz="0.0 0.0 0.0" rpy="0.0 0.0 0.0"/>
+          <parent link="${sequence}_finger_link_${finger_num*4+1}" />
+          <child link="${sequence}_finger_link_${finger_num*4+1}_cover" />
         </joint>
       </xacro:if>
@@ -519,5 +569,5 @@
       </xacro:if>
       <joint name="${sequence}_finger_joint_${finger_num*4+1}" type="revolute">
-        <limit effort="0" velocity="0" lower="${-0.296+0.1}" upper="${1.71-0.1}" />
+        <limit effort="15" velocity="7" lower="${-0.296+0.1}" upper="${1.71-0.1}" />
         <axis xyz="0 1 0"/>
         <parent link="${sequence}_finger_link_${finger_num*4+0}"/>
@@ -535,12 +585,17 @@
             </xacro:if>
           </geometry>
-          <material name="black"/>
+          <material name="black" />
         </visual>
         <collision>
           <geometry>
-            <box size="${0.0196} ${0.0275} ${0.0384}"/>
-          </geometry>
-          <origin rpy="0 0 0" xyz="0 0 ${0.0384/2}"/>
+            <box size="${0.0196} ${0.0275} ${0.0540}"/>
+          </geometry>
+          <origin rpy="0 0 0" xyz="0 0 ${0.0540/2}"/>
         </collision>
+        <inertial><!-- TO FILL IN-->
+          <origin xyz="0.0 0.0 0.0" rpy="0.0 0.0 0.0"/>
+          <mass value="0.0"/>
+          <inertia ixx="0.0" ixy="0.0" ixz="0.0" iyy="0.0" iyz="0.0" izz="0.0"/>
+        </inertial>
       </link>
       <xacro:if value="${covers == 1}">
@@ -558,9 +613,14 @@
             <origin rpy="0 0 0" xyz="0 0 ${0.0514/2}"/>
           </collision>
+          <inertial><!-- TO FILL IN-->
+            <origin xyz="0.0 0.0 0.0" rpy="0.0 0.0 0.0"/>
+            <mass value="0.0"/>
+            <inertia ixx="0.0" ixy="0.0" ixz="0.0" iyy="0.0" iyz="0.0" izz="0.0"/>
+          </inertial>
         </link>
         <joint name="${sequence}_finger_link_${finger_num*4+2}_cover_joint" type="fixed">
-        <origin xyz="0.0 0.0 0.0" rpy="0.0 0.0 0.0"/>
-        <parent link="${sequence}_finger_link_${finger_num*4+2}" />
-        <child link="${sequence}_finger_link_${finger_num*4+2}_cover" />
+          <origin xyz="0.0 0.0 0.0" rpy="0.0 0.0 0.0"/>
+          <parent link="${sequence}_finger_link_${finger_num*4+2}" />
+          <child link="${sequence}_finger_link_${finger_num*4+2}_cover" />
         </joint>
       </xacro:if>
@@ -570,5 +630,5 @@
       <joint name="${sequence}_finger_joint_${finger_num*4+2}" type="revolute">
         <axis xyz="0 1 0"/>
-        <limit effort="0" velocity="0" lower="${-0.274+0.1}" upper="${1.809-0.1}" />
+        <limit effort="15" velocity="7" lower="${-0.274+0.1}" upper="${1.809-0.1}" />
         <parent link="${sequence}_finger_link_${finger_num*4+1}"/>
         <child link="${sequence}_finger_link_${finger_num*4+2}"/>
@@ -580,19 +640,24 @@
             <mesh filename="package://xela_models/mesh/allegro/link_3.0.STL" />
           </geometry>
-          <material name="black"/>
+          <material name="black" />
         </visual>
         <collision>
           <geometry>
-            <box size="${0.0196} ${0.0275} ${0.0387-0.0120}"/>
-          </geometry>
-          <origin rpy="0 0 0" xyz="0 0 ${(0.0387-0.0120)/2}"/>
+            <box size="${0.0196} ${0.0275} ${0.0384-0.0120}"/>
+          </geometry>
+          <origin rpy="0 0 0" xyz="0 0 ${(0.0384-0.0120)/2}"/>
         </collision>
+        <inertial><!-- TO FILL IN-->
+          <origin xyz="0.0 0.0 0.0" rpy="0.0 0.0 0.0"/>
+          <mass value="0.0"/>
+          <inertia ixx="0.0" ixy="0.0" ixz="0.0" iyy="0.0" iyz="0.0" izz="0.0"/>
+        </inertial>
       </link>
       <joint name="${sequence}_finger_joint_${finger_num*4+3}" type="revolute">
         <axis xyz="0 1 0"/>
-        <limit effort="0" velocity="0" lower="${-0.327+0.1}" upper="${1.718-0.1}" />
+        <limit effort="15" velocity="7" lower="${-0.327+0.1}" upper="${1.718-0.1}" />
         <parent link="${sequence}_finger_link_${finger_num*4+2}"/>
         <child link="${sequence}_finger_link_${finger_num*4+3}"/>
-        <origin xyz="0 0.0002 0.043"/>
+        <origin xyz="0 0.0 0.0384"/>
       </joint>
     <xacro:if value="${tip == 'flat'}">
@@ -612,7 +677,5 @@
             <mesh filename="package://xela_models/mesh/allegro/link_12.0_right.STL" />
           </geometry>
-          <material name="black">
-            <color rgba=".2 .2 .2 1"/>
-          </material>
+          <material name="grey" />
         </visual>
         <collision>
@@ -622,8 +685,13 @@
           <origin rpy="0 0 0" xyz="${-0.0358/2+0.0} ${.018/2} ${.029/2}"/>
         </collision>
+        <inertial><!-- TO FILL IN-->
+          <origin xyz="0.0 0.0 0.0" rpy="0.0 0.0 0.0"/>
+          <mass value="0.0"/>
+          <inertia ixx="0.0" ixy="0.0" ixz="0.0" iyy="0.0" iyz="0.0" izz="0.0"/>
+        </inertial>
       </link>
       <joint name="${sequence}_joint_${finger_num*4+0}" type="revolute">
         <axis xyz="-1 0 0"/>
-        <limit effort="0" velocity="0" lower="${0.363-0.1}" upper="${1.496-0.1}" />
+        <limit effort="15" velocity="7" lower="${0.363-0.1}" upper="${1.496-0.1}" />
         <parent link="${parent}"/>
         <child link="${sequence}_link_${finger_num*4+0}"/>
@@ -635,7 +703,5 @@
             <mesh filename="package://xela_models/mesh/allegro/link_13.0.STL" />
           </geometry>
-          <material name="black">
-            <color rgba=".2 .2 .2 1"/>
-          </material>
+          <material name="grey" />
         </visual>
         <collision>
@@ -645,4 +711,9 @@
           <origin rpy="0 0 0" xyz="0 0 ${0.0177/2}"/>
         </collision>
+        <inertial><!-- TO FILL IN-->
+          <origin xyz="0.0 0.0 0.0" rpy="0.0 0.0 0.0"/>
+          <mass value="0.0"/>
+          <inertia ixx="0.0" ixy="0.0" ixz="0.0" iyy="0.0" iyz="0.0" izz="0.0"/>
+        </inertial>
       </link>
       <xacro:if value="${covers == 1}">
@@ -660,14 +731,19 @@
             <origin rpy="0 0 0" xyz="0 0 0"/>
           </collision>
+          <inertial><!-- TO FILL IN-->
+            <origin xyz="0.0 0.0 0.0" rpy="0.0 0.0 0.0"/>
+            <mass value="0.0"/>
+            <inertia ixx="0.0" ixy="0.0" ixz="0.0" iyy="0.0" iyz="0.0" izz="0.0"/>
+          </inertial>
         </link>
         <joint name="${sequence}_link_${finger_num*4+1}_cover_joint" type="fixed">
-        <origin xyz="0.0 0.0 0.0" rpy="0.0 0.0 0.0"/>
-        <parent link="${sequence}_link_${finger_num*4+2}" />
-        <child link="${sequence}_link_${finger_num*4+1}_cover" />
+          <origin xyz="0.0 0.0 0.0" rpy="0.0 0.0 0.0"/>
+          <parent link="${sequence}_link_${finger_num*4+2}" />
+          <child link="${sequence}_link_${finger_num*4+1}_cover" />
         </joint>
       </xacro:if>
       <joint name="${sequence}_joint_${finger_num*4+1}" type="revolute">
         <axis xyz="0 0 1"/>
-        <limit effort="0" velocity="0" lower="${-0.205+0.1}" upper="${1.263-0.1}" />
+        <limit effort="15" velocity="7" lower="${-0.205+0.1}" upper="${1.263-0.1}" />
         <parent link="${sequence}_link_${finger_num*4+0}"/>
         <child link="${sequence}_link_${finger_num*4+1}"/>
@@ -684,6 +760,5 @@
             </xacro:if>
           </geometry>
-          <material name="black">
-          </material>
+          <material name="black" />
         </visual>
         <collision>
@@ -693,4 +768,9 @@
           <origin rpy="0 0 0" xyz="0 0 ${0.0514/2}"/>
         </collision>
+        <inertial><!-- TO FILL IN-->
+          <origin xyz="0.0 0.0 0.0" rpy="0.0 0.0 0.0"/>
+          <mass value="0.0"/>
+          <inertia ixx="0.0" ixy="0.0" ixz="0.0" iyy="0.0" iyz="0.0" izz="0.0"/>
+        </inertial>
       </link>
       <xacro:if value="${covers == 1}">
@@ -708,9 +788,14 @@
             <origin rpy="0 0 0" xyz="0 0 0"/>
           </collision>
+          <inertial><!-- TO FILL IN-->
+            <origin xyz="0.0 0.0 0.0" rpy="0.0 0.0 0.0"/>
+            <mass value="0.0"/>
+            <inertia ixx="0.0" ixy="0.0" ixz="0.0" iyy="0.0" iyz="0.0" izz="0.0"/>
+          </inertial>
         </link>
         <joint name="${sequence}_link_${finger_num*4+2}_cover_joint" type="fixed">
-        <origin xyz="0.0 0.0 0.0" rpy="0.0 0.0 0.0"/>
-        <parent link="${sequence}_link_${finger_num*4+3}" />
-        <child link="${sequence}_link_${finger_num*4+2}_cover" />
+          <origin xyz="0.0 0.0 0.0" rpy="0.0 0.0 0.0"/>
+          <parent link="${sequence}_link_${finger_num*4+3}" />
+          <child link="${sequence}_link_${finger_num*4+2}_cover" />
         </joint>
       </xacro:if>
@@ -720,5 +805,5 @@
       <joint name="${sequence}_joint_${finger_num*4+2}" type="revolute">
         <axis xyz="0 1 0"/>
-        <limit effort="0" velocity="0" lower="${-0.289+0.1}" upper="${1.744-0.1}" />
+        <limit effort="15" velocity="7" lower="${-0.289+0.1}" upper="${1.744-0.1}" />
         <parent link="${sequence}_link_${finger_num*4+1}"/>
         <child link="${sequence}_link_${finger_num*4+2}"/>
@@ -735,6 +820,5 @@
             </xacro:if>
           </geometry>
-        <material name="black">
-        </material>
+        <material name="black" />
         </visual>
         <collision>
@@ -744,4 +828,9 @@
           <origin rpy="0 0 0" xyz="0 0 ${(0.0543-0.0120)/2}"/>
         </collision>
+        <inertial><!-- TO FILL IN-->
+          <origin xyz="0.0 0.0 0.0" rpy="0.0 0.0 0.0"/>
+          <mass value="0.0"/>
+          <inertia ixx="0.0" ixy="0.0" ixz="0.0" iyy="0.0" iyz="0.0" izz="0.0"/>
+        </inertial>
       </link>
       <xacro:if value="${phalanges == 1}">
@@ -750,5 +839,5 @@
     <joint name="${sequence}_joint_${finger_num*4+3}" type="revolute">
       <axis xyz="0 1 0"/>
-      <limit effort="0" velocity="0" lower="${-0.262+0.1}" upper="${1.819-0.1}" />
+      <limit effort="15" velocity="7" lower="${-0.262+0.1}" upper="${1.819-0.1}" />
       <parent link="${sequence}_link_${finger_num*4+2}"/>
       <child link="${sequence}_link_${finger_num*4+3}"/>
