Commit message: 'Update 2109291204'

File: xela_models/urdf/ahrcpcpn.urdf (robot description, URDF)
Before this commit: robot allegro_hand_right, 45 links, 44 joints
Links:
- link 1_hitosashi_finger_finger_link_1: geometry collision box size=0.0196 0.0275 0.0164; visual mesh filename=package://xela_models/mesh/allegro/link_1.1.stl
- link 1_hitosashi_finger_finger_link_2: geometry collision box size=0.0196 0.0275 0.054; visual mesh filename=package://xela_models/mesh/allegro/link_2.1.stl
- link 1_hitosashi_finger_finger_link_3: geometry collision box size=0.0196 0.0275 0.026399999999999996; visual mesh filename=package://xela_models/mesh/allegro/link_3.0.STL
- link 1_kusuri_finger_finger_link_10: geometry collision box size=0.0196 0.0275 0.054; visual mesh filename=package://xela_models/mesh/allegro/link_2.1.stl
- link 1_kusuri_finger_finger_link_11: geometry collision box size=0.0196 0.0275 0.026399999999999996; visual mesh filename=package://xela_models/mesh/allegro/link_3.0.STL
- link 1_kusuri_finger_finger_link_9: geometry collision box size=0.0196 0.0275 0.0164; visual mesh filename=package://xela_models/mesh/allegro/link_1.1.stl
- link 1_naka_finger_finger_link_5: geometry collision box size=0.0196 0.0275 0.0164; visual mesh filename=package://xela_models/mesh/allegro/link_1.1.stl
- link 1_naka_finger_finger_link_6: geometry collision box size=0.0196 0.0275 0.054; visual mesh filename=package://xela_models/mesh/allegro/link_2.1.stl
- link 1_naka_finger_finger_link_7: geometry collision box size=0.0196 0.0275 0.026399999999999996; visual mesh filename=package://xela_models/mesh/allegro/link_3.0.STL
Joints:
- joint 1_hitosashi_finger_finger_joint_0: limit lower=-0.47 upper=0.47 effort=0 velocity=0 -> lower=-0.47 upper=0.47 effort=15 velocity=7
- joint 1_hitosashi_finger_finger_joint_1: limit lower=-0.19599999999999998 upper=1.6099999999999999 effort=0 velocity=0 -> lower=-0.19599999999999998 upper=1.6099999999999999 effort=15 velocity=7
- joint 1_hitosashi_finger_finger_joint_2: limit lower=-0.17400000000000002 upper=1.7089999999999999 effort=0 velocity=0 -> lower=-0.17400000000000002 upper=1.7089999999999999 effort=15 velocity=7
- joint 1_hitosashi_finger_finger_joint_3: limit lower=-0.227 upper=1.6179999999999999 effort=0 velocity=0 -> lower=-0.227 upper=1.6179999999999999 effort=15 velocity=7; origin xyz=0 0.0002 0.043 -> xyz=0 0.0 0.0384
- joint 1_kusuri_finger_finger_joint_10: limit lower=-0.17400000000000002 upper=1.7089999999999999 effort=0 velocity=0 -> lower=-0.17400000000000002 upper=1.7089999999999999 effort=15 velocity=7
- joint 1_kusuri_finger_finger_joint_11: limit lower=-0.227 upper=1.6179999999999999 effort=0 velocity=0 -> lower=-0.227 upper=1.6179999999999999 effort=15 velocity=7; origin xyz=0 0.0002 0.043 -> xyz=0 0.0 0.0384
- joint 1_kusuri_finger_finger_joint_8: limit lower=-0.47 upper=0.47 effort=0 velocity=0 -> lower=-0.47 upper=0.47 effort=15 velocity=7
- joint 1_kusuri_finger_finger_joint_9: limit lower=-0.19599999999999998 upper=1.6099999999999999 effort=0 velocity=0 -> lower=-0.19599999999999998 upper=1.6099999999999999 effort=15 velocity=7
- joint 1_naka_finger_finger_joint_4: limit lower=-0.47 upper=0.47 effort=0 velocity=0 -> lower=-0.47 upper=0.47 effort=15 velocity=7
- joint 1_naka_finger_finger_joint_5: limit lower=-0.19599999999999998 upper=1.6099999999999999 effort=0 velocity=0 -> lower=-0.19599999999999998 upper=1.6099999999999999 effort=15 velocity=7
- joint 1_naka_finger_finger_joint_6: limit lower=-0.17400000000000002 upper=1.7089999999999999 effort=0 velocity=0 -> lower=-0.17400000000000002 upper=1.7089999999999999 effort=15 velocity=7
- joint 1_naka_finger_finger_joint_7: limit lower=-0.227 upper=1.6179999999999999 effort=0 velocity=0 -> lower=-0.227 upper=1.6179999999999999 effort=15 velocity=7; origin xyz=0 0.0002 0.043 -> xyz=0 0.0 0.0384
- joint 1_oya_finger_joint_12: limit lower=0.263 upper=1.396 effort=0 velocity=0 -> lower=0.263 upper=1.396 effort=15 velocity=7
- joint 1_oya_finger_joint_13: limit lower=-0.10499999999999998 upper=1.1629999999999998 effort=0 velocity=0 -> lower=-0.10499999999999998 upper=1.1629999999999998 effort=15 velocity=7
- joint 1_oya_finger_joint_14: limit lower=-0.18899999999999997 upper=1.644 effort=0 velocity=0 -> lower=-0.18899999999999997 upper=1.644 effort=15 velocity=7
- joint 1_oya_finger_joint_15: limit lower=-0.162 upper=1.7189999999999999 effort=0 velocity=0 -> lower=-0.162 upper=1.7189999999999999 effort=15 velocity=7

File: xela_models/urdf/xela.xacro (robot description, xacro)
@@ -3,8 +3,8 @@
   <!-- Rviz colors -->
   <material name="black">
-    <color rgba="0.0 0.0 0.0 1.0"/>
+    <color rgba="0.2 0.2 0.2 1.0"/>
   </material>
   <material name="blue">
-    <color rgba="0.0 0.0 0.8 1.0"/>
+    <color rgba="0.2 0.2 0.8 1.0"/>
   </material>
   <material name="green">
@@ -12,5 +12,5 @@
   </material>
   <material name="grey">
-    <color rgba="0.2 0.2 0.2 1.0"/>
+    <color rgba="0.4 0.4 0.4 1.0"/>
   </material>
   <material name="orange">
@@ -118,9 +118,4 @@
         <material name="${col}"/>
       </visual>
-      <inertial><!-- TO FILL IN-->
-        <origin xyz="0.0 0.0 0.0" rpy="0.0 0.0 0.0"/>
-        <mass value="0.0"/>
-        <inertia ixx="0.0" ixy="0.0" ixz="0.0" iyy="0.0" iyz="0.0" izz="0.0"/>
-      </inertial>
     </link>
     <link name="${sequence}_aftf_sensorbase_base_link">
@@ -188,9 +183,4 @@
         <material name="${col}"/>
       </visual>
-      <inertial><!-- TO FILL IN-->
-        <origin xyz="0.0 0.0 0.0" rpy="0.0 0.0 0.0"/>
-        <mass value="0.0"/>
-        <inertia ixx="0.0" ixy="0.0" ixz="0.0" iyy="0.0" iyz="0.0" izz="0.0"/>
-      </inertial>
     </link>
     <xacro:if value="${taxels == 1}">
@@ -247,9 +237,4 @@
         <material name="${col}"/>
       </visual>
-      <inertial><!-- TO FILL IN (Allegro defaults)-->
-        <origin xyz="0.0 0.0 0.0" rpy="0.0 0.0 0.0"/>
-        <mass value="0.0"/>
-        <inertia ixx="0.0" ixy="0.0" ixz="0.0" iyy="0.0" iyz="0.0" izz="0.0"/>
-      </inertial>
     </link>
   </xacro:macro>
@@ -276,9 +261,4 @@
         </visual>
       </xacro:if>
-      <inertial><!-- TO FILL IN-->
-        <origin xyz="0.0 0.0 0.0" rpy="0.0 0.0 0.0"/>
-        <mass value="0.0"/>
-        <inertia ixx="0.0" ixy="0.0" ixz="0.0" iyy="0.0" iyz="0.0" izz="0.0"/>
-      </inertial>
     </link>
     <xacro:if value="${taxels == 1}">
@@ -323,9 +303,4 @@
         </visual>
       </xacro:if>
-      <inertial><!-- TO FILL IN-->
-        <origin xyz="0.0 0.0 0.0" rpy="0.0 0.0 0.0"/>
-        <mass value="0.0"/>
-        <inertia ixx="0.0" ixy="0.0" ixz="0.0" iyy="0.0" iyz="0.0" izz="0.0"/>
-      </inertial>
     </link>
     <xacro:if value="${taxels == 1}">
@@ -360,9 +335,4 @@
         </visual>
       </xacro:if>
-      <inertial><!-- TO FILL IN-->
-        <origin xyz="0.0 0.0 0.0" rpy="0.0 0.0 0.0"/>
-        <mass value="0.0"/>
-        <inertia ixx="0.0" ixy="0.0" ixz="0.0" iyy="0.0" iyz="0.0" izz="0.0"/>
-      </inertial>
     </link>
     <xacro:if value="${taxels == 1}">
@@ -416,9 +386,4 @@
         </geometry>
       </collision>
-      <inertial><!-- TO FILL IN BASE-->
-        <origin xyz="0.0 0.0 0.0" rpy="0.0 0.0 0.0"/>
-        <mass value="0.0"/>
-        <inertia ixx="0.0" ixy="0.0" ixz="0.0" iyy="0.0" iyz="0.0" izz="0.0"/>
-      </inertial>
     </link>
     <joint name="${sequence}_ahr_fixed" type="fixed">
@@ -501,9 +466,4 @@
           <origin rpy="0 0 0" xyz="0 0 ${0.0164/2+0.003}"/>
         </collision>
-        <inertial><!-- TO FILL IN-->
-          <origin xyz="0.0 0.0 0.0" rpy="0.0 0.0 0.0"/>
-          <mass value="0.0"/>
-          <inertia ixx="0.0" ixy="0.0" ixz="0.0" iyy="0.0" iyz="0.0" izz="0.0"/>
-        </inertial>
       </link>
       <joint name="${sequence}_finger_joint_${finger_num*4+0}" type="revolute">
@@ -532,9 +492,4 @@
           <origin rpy="0 0 0" xyz="0 0 ${0.0164/2}"/>
         </collision>
-        <inertial><!-- TO FILL IN-->
-          <origin xyz="0.0 0.0 0.0" rpy="0.0 0.0 0.0"/>
-          <mass value="0.0"/>
-          <inertia ixx="0.0" ixy="0.0" ixz="0.0" iyy="0.0" iyz="0.0" izz="0.0"/>
-        </inertial>
       </link>
       <xacro:if value="${covers == 1}">
@@ -552,9 +507,4 @@
             <origin rpy="0 0 0" xyz="0 0 ${0.0177/2}"/>
           </collision>
-          <inertial><!-- TO FILL IN-->
-            <origin xyz="0.0 0.0 0.0" rpy="0.0 0.0 0.0"/>
-            <mass value="0.0"/>
-            <inertia ixx="0.0" ixy="0.0" ixz="0.0" iyy="0.0" iyz="0.0" izz="0.0"/>
-          </inertial>
         </link>
         <joint name="${sequence}_finger_link_${finger_num*4+1}_cover_joint" type="fixed">
@@ -593,9 +543,4 @@
           <origin rpy="0 0 0" xyz="0 0 ${0.0540/2}"/>
         </collision>
-        <inertial><!-- TO FILL IN-->
-          <origin xyz="0.0 0.0 0.0" rpy="0.0 0.0 0.0"/>
-          <mass value="0.0"/>
-          <inertia ixx="0.0" ixy="0.0" ixz="0.0" iyy="0.0" iyz="0.0" izz="0.0"/>
-        </inertial>
       </link>
       <xacro:if value="${covers == 1}">
@@ -613,9 +558,4 @@
             <origin rpy="0 0 0" xyz="0 0 ${0.0514/2}"/>
           </collision>
-          <inertial><!-- TO FILL IN-->
-            <origin xyz="0.0 0.0 0.0" rpy="0.0 0.0 0.0"/>
-            <mass value="0.0"/>
-            <inertia ixx="0.0" ixy="0.0" ixz="0.0" iyy="0.0" iyz="0.0" izz="0.0"/>
-          </inertial>
         </link>
         <joint name="${sequence}_finger_link_${finger_num*4+2}_cover_joint" type="fixed">
@@ -648,9 +588,4 @@
           <origin rpy="0 0 0" xyz="0 0 ${(0.0384-0.0120)/2}"/>
         </collision>
-        <inertial><!-- TO FILL IN-->
-          <origin xyz="0.0 0.0 0.0" rpy="0.0 0.0 0.0"/>
-          <mass value="0.0"/>
-          <inertia ixx="0.0" ixy="0.0" ixz="0.0" iyy="0.0" iyz="0.0" izz="0.0"/>
-        </inertial>
       </link>
       <joint name="${sequence}_finger_joint_${finger_num*4+3}" type="revolute">
@@ -685,9 +620,4 @@
           <origin rpy="0 0 0" xyz="${-0.0358/2+0.0} ${.018/2} ${.029/2}"/>
         </collision>
-        <inertial><!-- TO FILL IN-->
-          <origin xyz="0.0 0.0 0.0" rpy="0.0 0.0 0.0"/>
-          <mass value="0.0"/>
-          <inertia ixx="0.0" ixy="0.0" ixz="0.0" iyy="0.0" iyz="0.0" izz="0.0"/>
-        </inertial>
       </link>
       <joint name="${sequence}_joint_${finger_num*4+0}" type="revolute">
@@ -711,9 +641,4 @@
           <origin rpy="0 0 0" xyz="0 0 ${0.0177/2}"/>
         </collision>
-        <inertial><!-- TO FILL IN-->
-          <origin xyz="0.0 0.0 0.0" rpy="0.0 0.0 0.0"/>
-          <mass value="0.0"/>
-          <inertia ixx="0.0" ixy="0.0" ixz="0.0" iyy="0.0" iyz="0.0" izz="0.0"/>
-        </inertial>
       </link>
       <xacro:if value="${covers == 1}">
@@ -731,9 +656,4 @@
             <origin rpy="0 0 0" xyz="0 0 0"/>
           </collision>
-          <inertial><!-- TO FILL IN-->
-            <origin xyz="0.0 0.0 0.0" rpy="0.0 0.0 0.0"/>
-            <mass value="0.0"/>
-            <inertia ixx="0.0" ixy="0.0" ixz="0.0" iyy="0.0" iyz="0.0" izz="0.0"/>
-          </inertial>
         </link>
         <joint name="${sequence}_link_${finger_num*4+1}_cover_joint" type="fixed">
@@ -768,9 +688,4 @@
           <origin rpy="0 0 0" xyz="0 0 ${0.0514/2}"/>
         </collision>
-        <inertial><!-- TO FILL IN-->
-          <origin xyz="0.0 0.0 0.0" rpy="0.0 0.0 0.0"/>
-          <mass value="0.0"/>
-          <inertia ixx="0.0" ixy="0.0" ixz="0.0" iyy="0.0" iyz="0.0" izz="0.0"/>
-        </inertial>
       </link>
       <xacro:if value="${covers == 1}">
@@ -788,9 +703,4 @@
             <origin rpy="0 0 0" xyz="0 0 0"/>
           </collision>
-          <inertial><!-- TO FILL IN-->
-            <origin xyz="0.0 0.0 0.0" rpy="0.0 0.0 0.0"/>
-            <mass value="0.0"/>
-            <inertia ixx="0.0" ixy="0.0" ixz="0.0" iyy="0.0" iyz="0.0" izz="0.0"/>
-          </inertial>
         </link>
         <joint name="${sequence}_link_${finger_num*4+2}_cover_joint" type="fixed">
@@ -828,9 +738,4 @@
           <origin rpy="0 0 0" xyz="0 0 ${(0.0543-0.0120)/2}"/>
         </collision>
-        <inertial><!-- TO FILL IN-->
-          <origin xyz="0.0 0.0 0.0" rpy="0.0 0.0 0.0"/>
-          <mass value="0.0"/>
-          <inertia ixx="0.0" ixy="0.0" ixz="0.0" iyy="0.0" iyz="0.0" izz="0.0"/>
-        </inertial>
       </link>
       <xacro:if value="${phalanges == 1}">
