Commit message: 'Update 2110041600'

File: xela_models/urdf/ahrcpcpn.urdf (robot description, URDF)
Before this commit: robot allegro_hand_right, 45 links, 44 joints
Links:
- removed link 1_ahr_base_link
- removed link 1_ahr_palm_1_4x6_base_link
- removed link 1_ahr_palm_2_4x6_base_link
- removed link 1_ahr_palm_3_4x6_base_link
- removed link 1_hitosashi_finger_finger_0_aftc_base_link
- removed link 1_hitosashi_finger_finger_link_0
- removed link 1_hitosashi_finger_finger_link_1
- removed link 1_hitosashi_finger_finger_link_1A_4x4_base_link
- removed link 1_hitosashi_finger_finger_link_1B_4x4_base_link
- removed link 1_hitosashi_finger_finger_link_1_cover
- removed link 1_hitosashi_finger_finger_link_2
- removed link 1_hitosashi_finger_finger_link_2_4x4_base_link
- removed link 1_hitosashi_finger_finger_link_2_cover
- removed link 1_hitosashi_finger_finger_link_3
- removed link 1_kusuri_finger_finger_2_aftc_base_link
- removed link 1_kusuri_finger_finger_link_10
- removed link 1_kusuri_finger_finger_link_10_4x4_base_link
- removed link 1_kusuri_finger_finger_link_10_cover
- removed link 1_kusuri_finger_finger_link_11
- removed link 1_kusuri_finger_finger_link_8
- removed link 1_kusuri_finger_finger_link_9
- removed link 1_kusuri_finger_finger_link_9A_4x4_base_link
- removed link 1_kusuri_finger_finger_link_9B_4x4_base_link
- removed link 1_kusuri_finger_finger_link_9_cover
- removed link 1_naka_finger_finger_1_aftc_base_link
- removed link 1_naka_finger_finger_link_4
- removed link 1_naka_finger_finger_link_5
- removed link 1_naka_finger_finger_link_5A_4x4_base_link
- removed link 1_naka_finger_finger_link_5B_4x4_base_link
- removed link 1_naka_finger_finger_link_5_cover
- removed link 1_naka_finger_finger_link_6
- removed link 1_naka_finger_finger_link_6_4x4_base_link
- removed link 1_naka_finger_finger_link_6_cover
- removed link 1_naka_finger_finger_link_7
- removed link 1_oya_finger_3_aftc_base_link
- removed link 1_oya_finger_link_12
- removed link 1_oya_finger_link_13
- removed link 1_oya_finger_link_13_cover
- removed link 1_oya_finger_link_14
- removed link 1_oya_finger_link_14_4x4_base_link
- removed link 1_oya_finger_link_14_cover
- removed link 1_oya_finger_link_15
- removed link 1_oya_finger_link_15_4x4_base_link
- added link ahr_palm_1_4x6_base_link; collision mesh filename=package://xela_models/mesh/4x6.stl; visual mesh filename=package://xela_models/mesh/4x6.stl
- added link ahr_palm_2_4x6_base_link; collision mesh filename=package://xela_models/mesh/4x6.stl; visual mesh filename=package://xela_models/mesh/4x6.stl
- added link ahr_palm_3_4x6_base_link; collision mesh filename=package://xela_models/mesh/4x6.stl; visual mesh filename=package://xela_models/mesh/4x6.stl
- added link hitosashi_finger_finger_0_aftc_base_link; collision mesh filename=package://xela_models/mesh/ft_c_collision.stl; visual mesh filename=package://xela_models/mesh/ft_c_visual.stl
- added link hitosashi_finger_finger_link_0, mass 0.0127; collision box size=0.0196 0.0275 0.0164; visual mesh filename=package://xela_models/mesh/allegro/link_0.0_ext.STL
- added link hitosashi_finger_finger_link_1, mass 0.0809; collision box size=0.0196 0.0275 0.0164; visual mesh filename=package://xela_models/mesh/allegro/link_1.1.stl
- added link hitosashi_finger_finger_link_1A_4x4_base_link; collision mesh filename=package://xela_models/mesh/4x4.stl
- added link hitosashi_finger_finger_link_1B_4x4_base_link; collision mesh filename=package://xela_models/mesh/4x4.stl
- added link hitosashi_finger_finger_link_1_cover; collision mesh filename=package://xela_models/mesh/allegro/link_1_cover.stl; visual mesh filename=package://xela_models/mesh/allegro/link_1_cover.stl
- added link hitosashi_finger_finger_link_2, mass 0.0447; collision box size=0.0196 0.0275 0.054; visual mesh filename=package://xela_models/mesh/allegro/link_2.1.stl
- added link hitosashi_finger_finger_link_2_4x4_base_link; collision mesh filename=package://xela_models/mesh/4x4.stl
- added link hitosashi_finger_finger_link_2_cover; collision mesh filename=package://xela_models/mesh/allegro/link_2_cover.stl; visual mesh filename=package://xela_models/mesh/allegro/link_2_cover.stl
- added link hitosashi_finger_finger_link_3, mass 0.0404; collision box size=0.0196 0.0275 0.026399999999999996; visual mesh filename=package://xela_models/mesh/allegro/link_3.0.STL
- added link kusuri_finger_finger_2_aftc_base_link; collision mesh filename=package://xela_models/mesh/ft_c_collision.stl; visual mesh filename=package://xela_models/mesh/ft_c_visual.stl
- added link kusuri_finger_finger_link_10, mass 0.0447; collision box size=0.0196 0.0275 0.054; visual mesh filename=package://xela_models/mesh/allegro/link_2.1.stl
- added link kusuri_finger_finger_link_10_4x4_base_link; collision mesh filename=package://xela_models/mesh/4x4.stl
- added link kusuri_finger_finger_link_10_cover; collision mesh filename=package://xela_models/mesh/allegro/link_2_cover.stl; visual mesh filename=package://xela_models/mesh/allegro/link_2_cover.stl
- added link kusuri_finger_finger_link_11, mass 0.0404; collision box size=0.0196 0.0275 0.026399999999999996; visual mesh filename=package://xela_models/mesh/allegro/link_3.0.STL
- added link kusuri_finger_finger_link_8, mass 0.0127; collision box size=0.0196 0.0275 0.0164; visual mesh filename=package://xela_models/mesh/allegro/link_0.0_ext.STL
- added link kusuri_finger_finger_link_9, mass 0.0809; collision box size=0.0196 0.0275 0.0164; visual mesh filename=package://xela_models/mesh/allegro/link_1.1.stl
- added link kusuri_finger_finger_link_9A_4x4_base_link; collision mesh filename=package://xela_models/mesh/4x4.stl
- added link kusuri_finger_finger_link_9B_4x4_base_link; collision mesh filename=package://xela_models/mesh/4x4.stl
- added link kusuri_finger_finger_link_9_cover; collision mesh filename=package://xela_models/mesh/allegro/link_1_cover.stl; visual mesh filename=package://xela_models/mesh/allegro/link_1_cover.stl
- added link naka_finger_finger_1_aftc_base_link; collision mesh filename=package://xela_models/mesh/ft_c_collision.stl; visual mesh filename=package://xela_models/mesh/ft_c_visual.stl
- added link naka_finger_finger_link_4, mass 0.0127; collision box size=0.0196 0.0275 0.0164; visual mesh filename=package://xela_models/mesh/allegro/link_0.0_ext.STL
- added link naka_finger_finger_link_5, mass 0.0809; collision box size=0.0196 0.0275 0.0164; visual mesh filename=package://xela_models/mesh/allegro/link_1.1.stl
- added link naka_finger_finger_link_5A_4x4_base_link; collision mesh filename=package://xela_models/mesh/4x4.stl
- added link naka_finger_finger_link_5B_4x4_base_link; collision mesh filename=package://xela_models/mesh/4x4.stl
- added link naka_finger_finger_link_5_cover; collision mesh filename=package://xela_models/mesh/allegro/link_1_cover.stl; visual mesh filename=package://xela_models/mesh/allegro/link_1_cover.stl
- added link naka_finger_finger_link_6, mass 0.0447; collision box size=0.0196 0.0275 0.054; visual mesh filename=package://xela_models/mesh/allegro/link_2.1.stl
- added link naka_finger_finger_link_6_4x4_base_link; collision mesh filename=package://xela_models/mesh/4x4.stl
- added link naka_finger_finger_link_6_cover; collision mesh filename=package://xela_models/mesh/allegro/link_2_cover.stl; visual mesh filename=package://xela_models/mesh/allegro/link_2_cover.stl
- added link naka_finger_finger_link_7, mass 0.0404; collision box size=0.0196 0.0275 0.026399999999999996; visual mesh filename=package://xela_models/mesh/allegro/link_3.0.STL
- added link oya_finger_3_aftc_base_link; collision mesh filename=package://xela_models/mesh/ft_c_collision.stl; visual mesh filename=package://xela_models/mesh/ft_c_visual.stl
- added link oya_finger_link_12, mass 0.0176; collision box size=0.0358 0.034 0.0455; visual mesh filename=package://xela_models/mesh/allegro/link_12.0_right.STL
- added link oya_finger_link_13, mass 0.0127; collision box size=0.0196 0.0275 0.0177; visual mesh filename=package://xela_models/mesh/allegro/link_13.0.STL
- added link oya_finger_link_14, mass 0.0457; collision box size=0.0196 0.0275 0.0514; visual mesh filename=package://xela_models/mesh/allegro/thumb_1.1.stl
- added link oya_finger_link_14_4x4_base_link; collision mesh filename=package://xela_models/mesh/4x4.stl
- added link oya_finger_link_14_cover; collision mesh filename=package://xela_models/mesh/allegro/thumb_1_cover.stl; visual mesh filename=package://xela_models/mesh/allegro/thumb_1_cover.stl
- added link oya_finger_link_15, mass 0.0753; collision box size=0.0196 0.0275 0.042300000000000004; visual mesh filename=package://xela_models/mesh/allegro/thumb_2.1.stl
- added link oya_finger_link_15_4x4_base_link; collision mesh filename=package://xela_models/mesh/4x4.stl
- added link oya_finger_link_15_cover; collision mesh filename=package://xela_models/mesh/allegro/thumb_2_cover.stl; visual mesh filename=package://xela_models/mesh/allegro/thumb_2_cover.stl
- link base_link: mass None -> 0.4288; geometry collision box size=0.0408 0.1130 0.095; visual mesh filename=package://xela_models/mesh/allegro/base.stl
Joints:
- removed joint 1_ahr_fixed
- removed joint 1_ahr_palm_1_4x6_fixed
- removed joint 1_ahr_palm_2_4x6_fixed
- removed joint 1_ahr_palm_3_4x6_fixed
- removed joint 1_hitosashi_finger_finger_0_aftc_fixed
- removed joint 1_hitosashi_finger_finger_joint_0
- removed joint 1_hitosashi_finger_finger_joint_1
- removed joint 1_hitosashi_finger_finger_joint_2
- removed joint 1_hitosashi_finger_finger_joint_3
- removed joint 1_hitosashi_finger_finger_link_1A_4x4_fixed
- removed joint 1_hitosashi_finger_finger_link_1B_4x4_fixed
- removed joint 1_hitosashi_finger_finger_link_1_cover_joint
- removed joint 1_hitosashi_finger_finger_link_2_4x4_fixed
- removed joint 1_hitosashi_finger_finger_link_2_cover_joint
- removed joint 1_kusuri_finger_finger_2_aftc_fixed
- removed joint 1_kusuri_finger_finger_joint_10
- removed joint 1_kusuri_finger_finger_joint_11
- removed joint 1_kusuri_finger_finger_joint_8
- removed joint 1_kusuri_finger_finger_joint_9
- removed joint 1_kusuri_finger_finger_link_10_4x4_fixed
- removed joint 1_kusuri_finger_finger_link_10_cover_joint
- removed joint 1_kusuri_finger_finger_link_9A_4x4_fixed
- removed joint 1_kusuri_finger_finger_link_9B_4x4_fixed
- removed joint 1_kusuri_finger_finger_link_9_cover_joint
- removed joint 1_naka_finger_finger_1_aftc_fixed
- removed joint 1_naka_finger_finger_joint_4
- removed joint 1_naka_finger_finger_joint_5
- removed joint 1_naka_finger_finger_joint_6
- removed joint 1_naka_finger_finger_joint_7
- removed joint 1_naka_finger_finger_link_5A_4x4_fixed
- removed joint 1_naka_finger_finger_link_5B_4x4_fixed
- removed joint 1_naka_finger_finger_link_5_cover_joint
- removed joint 1_naka_finger_finger_link_6_4x4_fixed
- removed joint 1_naka_finger_finger_link_6_cover_joint
- removed joint 1_oya_finger_3_aftc_fixed
- removed joint 1_oya_finger_joint_12
- removed joint 1_oya_finger_joint_13
- removed joint 1_oya_finger_joint_14
- removed joint 1_oya_finger_joint_15
- removed joint 1_oya_finger_link_13_cover_joint
- removed joint 1_oya_finger_link_14_4x4_fixed
- removed joint 1_oya_finger_link_14_cover_joint
- removed joint 1_oya_finger_link_15_4x4_fixed
- removed joint fixed
- added joint ahr_fixed: type fixed, parent world, child base_link, origin xyz=0.0 0.0 0.0 rpy=0.0 0.0 0.0
- added joint ahr_palm_1_4x6_fixed: type fixed, parent base_link, child ahr_palm_1_4x6_base_link, origin xyz=0.013 -0.051 -0.0365 rpy=1.5707963267948966 0.0 1.5707963267948966
- added joint ahr_palm_2_4x6_fixed: type fixed, parent base_link, child ahr_palm_2_4x6_base_link, origin xyz=0.013 0.0523 -0.005 rpy=1.5707963267948966 3.141592653589793 1.5707963267948966
- added joint ahr_palm_3_4x6_fixed: type fixed, parent base_link, child ahr_palm_3_4x6_base_link, origin xyz=0.013 -0.051 -0.068 rpy=1.5707963267948966 0.0 1.5707963267948966
- added joint hitosashi_finger_finger_0_aftc_fixed: type fixed, parent hitosashi_finger_finger_link_3, child hitosashi_finger_finger_0_aftc_base_link, origin xyz=-0.013 0.0 0.016 rpy=1.5707963267948966 0.0 1.5707963267948966
- added joint hitosashi_finger_finger_joint_0: type revolute, parent base_link, child hitosashi_finger_finger_link_0, origin xyz=0 0.0435 -0.001542 rpy=-0.08726646259971647 0 0, axis 0 0 1, limit lower=-0.47 upper=0.47 effort=15 velocity=7
- added joint hitosashi_finger_finger_joint_1: type revolute, parent hitosashi_finger_finger_link_0, child hitosashi_finger_finger_link_1, origin xyz=0 0 0.0204, axis 0 1 0, limit lower=-0.19599999999999998 upper=1.6099999999999999 effort=15 velocity=7
- added joint hitosashi_finger_finger_joint_2: type revolute, parent hitosashi_finger_finger_link_1, child hitosashi_finger_finger_link_2, origin xyz=0 0 0.054, axis 0 1 0, limit lower=-0.17400000000000002 upper=1.7089999999999999 effort=15 velocity=7
- added joint hitosashi_finger_finger_joint_3: type revolute, parent hitosashi_finger_finger_link_2, child hitosashi_finger_finger_link_3, origin xyz=0 0.0 0.0384, axis 0 1 0, limit lower=-0.227 upper=1.6179999999999999 effort=15 velocity=7
- added joint hitosashi_finger_finger_link_1A_4x4_fixed: type fixed, parent hitosashi_finger_finger_link_1, child hitosashi_finger_finger_link_1A_4x4_base_link, origin xyz=0.0108 0.012 0.033 rpy=0.0 -1.5707963267948966 3.141592653589793
- added joint hitosashi_finger_finger_link_1B_4x4_fixed: type fixed, parent hitosashi_finger_finger_link_1, child hitosashi_finger_finger_link_1B_4x4_base_link, origin xyz=0.0108 -0.012 0.021 rpy=0.0 1.5707963267948966 0.0
- added joint hitosashi_finger_finger_link_1_cover_joint: type fixed, parent hitosashi_finger_finger_link_1, child hitosashi_finger_finger_link_1_cover, origin xyz=0.0 0.0 0.0 rpy=0.0 0.0 0.0
- added joint hitosashi_finger_finger_link_2_4x4_fixed: type fixed, parent hitosashi_finger_finger_link_2, child hitosashi_finger_finger_link_2_4x4_base_link, origin xyz=0.01 -0.012 0.0445 rpy=0.0 1.5707963267948966 0.0
- added joint hitosashi_finger_finger_link_2_cover_joint: type fixed, parent hitosashi_finger_finger_link_2, child hitosashi_finger_finger_link_2_cover, origin xyz=0.0 0.0 0.0 rpy=0.0 0.0 0.0
- added joint kusuri_finger_finger_2_aftc_fixed: type fixed, parent kusuri_finger_finger_link_11, child kusuri_finger_finger_2_aftc_base_link, origin xyz=-0.013 0.0 0.016 rpy=1.5707963267948966 0.0 1.5707963267948966
- added joint kusuri_finger_finger_joint_10: type revolute, parent kusuri_finger_finger_link_9, child kusuri_finger_finger_link_10, origin xyz=0 0 0.054, axis 0 1 0, limit lower=-0.17400000000000002 upper=1.7089999999999999 effort=15 velocity=7
- added joint kusuri_finger_finger_joint_11: type revolute, parent kusuri_finger_finger_link_10, child kusuri_finger_finger_link_11, origin xyz=0 0.0 0.0384, axis 0 1 0, limit lower=-0.227 upper=1.6179999999999999 effort=15 velocity=7
- added joint kusuri_finger_finger_joint_8: type revolute, parent base_link, child kusuri_finger_finger_link_8, origin xyz=0 -0.0435 -0.001542 rpy=0.08726646259971647 0 0, axis 0 0 1, limit lower=-0.47 upper=0.47 effort=15 velocity=7
- added joint kusuri_finger_finger_joint_9: type revolute, parent kusuri_finger_finger_link_8, child kusuri_finger_finger_link_9, origin xyz=0 0 0.0204, axis 0 1 0, limit lower=-0.19599999999999998 upper=1.6099999999999999 effort=15 velocity=7
- added joint kusuri_finger_finger_link_10_4x4_fixed: type fixed, parent kusuri_finger_finger_link_10, child kusuri_finger_finger_link_10_4x4_base_link, origin xyz=0.01 -0.012 0.0445 rpy=0.0 1.5707963267948966 0.0
- added joint kusuri_finger_finger_link_10_cover_joint: type fixed, parent kusuri_finger_finger_link_10, child kusuri_finger_finger_link_10_cover, origin xyz=0.0 0.0 0.0 rpy=0.0 0.0 0.0
- added joint kusuri_finger_finger_link_9A_4x4_fixed: type fixed, parent kusuri_finger_finger_link_9, child kusuri_finger_finger_link_9A_4x4_base_link, origin xyz=0.0108 0.012 0.033 rpy=0.0 -1.5707963267948966 3.141592653589793
- added joint kusuri_finger_finger_link_9B_4x4_fixed: type fixed, parent kusuri_finger_finger_link_9, child kusuri_finger_finger_link_9B_4x4_base_link, origin xyz=0.0108 -0.012 0.021 rpy=0.0 1.5707963267948966 0.0
- added joint kusuri_finger_finger_link_9_cover_joint: type fixed, parent kusuri_finger_finger_link_9, child kusuri_finger_finger_link_9_cover, origin xyz=0.0 0.0 0.0 rpy=0.0 0.0 0.0
- added joint naka_finger_finger_1_aftc_fixed: type fixed, parent naka_finger_finger_link_7, child naka_finger_finger_1_aftc_base_link, origin xyz=-0.013 0.0 0.016 rpy=1.5707963267948966 0.0 1.5707963267948966
- added joint naka_finger_finger_joint_4: type revolute, parent base_link, child naka_finger_finger_link_4, origin xyz=0 0 0.0007 rpy=0.0 0 0, axis 0 0 1, limit lower=-0.47 upper=0.47 effort=15 velocity=7
- added joint naka_finger_finger_joint_5: type revolute, parent naka_finger_finger_link_4, child naka_finger_finger_link_5, origin xyz=0 0 0.0204, axis 0 1 0, limit lower=-0.19599999999999998 upper=1.6099999999999999 effort=15 velocity=7
- added joint naka_finger_finger_joint_6: type revolute, parent naka_finger_finger_link_5, child naka_finger_finger_link_6, origin xyz=0 0 0.054, axis 0 1 0, limit lower=-0.17400000000000002 upper=1.7089999999999999 effort=15 velocity=7
- added joint naka_finger_finger_joint_7: type revolute, parent naka_finger_finger_link_6, child naka_finger_finger_link_7, origin xyz=0 0.0 0.0384, axis 0 1 0, limit lower=-0.227 upper=1.6179999999999999 effort=15 velocity=7
- added joint naka_finger_finger_link_5A_4x4_fixed: type fixed, parent naka_finger_finger_link_5, child naka_finger_finger_link_5A_4x4_base_link, origin xyz=0.0108 0.012 0.033 rpy=0.0 -1.5707963267948966 3.141592653589793
- added joint naka_finger_finger_link_5B_4x4_fixed: type fixed, parent naka_finger_finger_link_5, child naka_finger_finger_link_5B_4x4_base_link, origin xyz=0.0108 -0.012 0.021 rpy=0.0 1.5707963267948966 0.0
- added joint naka_finger_finger_link_5_cover_joint: type fixed, parent naka_finger_finger_link_5, child naka_finger_finger_link_5_cover, origin xyz=0.0 0.0 0.0 rpy=0.0 0.0 0.0
- added joint naka_finger_finger_link_6_4x4_fixed: type fixed, parent naka_finger_finger_link_6, child naka_finger_finger_link_6_4x4_base_link, origin xyz=0.01 -0.012 0.0445 rpy=0.0 1.5707963267948966 0.0
- added joint naka_finger_finger_link_6_cover_joint: type fixed, parent naka_finger_finger_link_6, child naka_finger_finger_link_6_cover, origin xyz=0.0 0.0 0.0 rpy=0.0 0.0 0.0
- added joint oya_finger_3_aftc_fixed: type fixed, parent oya_finger_link_15, child oya_finger_3_aftc_base_link, origin xyz=-0.013 0.0 0.0315 rpy=1.5707963267948966 0.0 1.5707963267948966
- added joint oya_finger_joint_12: type revolute, parent base_link, child oya_finger_link_12, origin xyz=-0.0182 0.019333 -0.045987 rpy=0 -1.6580627893946132 -1.5707963267948966, axis -1 0 0, limit lower=0.263 upper=1.396 effort=15 velocity=7
- added joint oya_finger_joint_13: type revolute, parent oya_finger_link_12, child oya_finger_link_13, origin xyz=-0.027 0.005 0.0399, axis 0 0 1, limit lower=-0.10499999999999998 upper=1.1629999999999998 effort=15 velocity=7
- added joint oya_finger_joint_14: type revolute, parent oya_finger_link_13, child oya_finger_link_14, origin xyz=0 0 0.0177, axis 0 1 0, limit lower=-0.18899999999999997 upper=1.644 effort=15 velocity=7
- added joint oya_finger_joint_15: type revolute, parent oya_finger_link_14, child oya_finger_link_15, origin xyz=0 0 0.0514, axis 0 1 0, limit lower=-0.162 upper=1.7189999999999999 effort=15 velocity=7
- added joint oya_finger_link_14_4x4_fixed: type fixed, parent oya_finger_link_14, child oya_finger_link_14_4x4_base_link, origin xyz=0.011 -0.012 0.023 rpy=0.0 1.5707963267948966 0.0
- added joint oya_finger_link_14_cover_joint: type fixed, parent oya_finger_link_14, child oya_finger_link_14_cover, origin xyz=0.0 0.0 0.0 rpy=0.0 0.0 0.0
- added joint oya_finger_link_15_4x4_fixed: type fixed, parent oya_finger_link_15, child oya_finger_link_15_4x4_base_link, origin xyz=0.011 -0.012 0.021 rpy=0.0 1.5707963267948966 0.0
- added joint oya_finger_link_15_cover_joint: type fixed, parent oya_finger_link_15, child oya_finger_link_15_cover, origin xyz=0.0 0.0 0.0 rpy=0.0 0.0 0.0

File: xela_models/urdf/allegro_hand_right.xacro (robot description, xacro)
@@ -4,22 +4,4 @@
 <xacro:include filename="$(find xela_models)/urdf/xela.xacro" />
 <link name="world" />
-<!--
-<joint name="fixed" type="fixed">
-    <parent link="world" />
-    <child link="base_link" />
-  </joint>
-  <link name="base_link">
-    <visual>
-      <geometry>
-        <sphere radius="0.001"/>
-      </geometry>
-      <origin xyz="0.0 0.0 0.0" rpy="0 0 0"/>
-    </visual>
-    <collision>
-      <geometry>
-        <sphere radius="0.001"/>
-      </geometry>
-    </collision>
-  </link> -->
 <!-- Notes
 Back controller covers can be disabled by setting covers to 0
@@ -27,7 +9,7 @@
 Palm sensors can be disabled by setting palm to 0
 -->
-	<xacro:allegro_hand_right sequence="1" tips="curved" parent="world" />
+	<xacro:allegro_hand_right sequence="" tips="curved" parent="world" />
   <!-- Enable the following 2 if you would like to see different options the same time -->
-	<!-- <xacro:allegro_hand_right sequence="2" parent="base_link" x="0.2" tips="curved" /> -->
-	<!-- <xacro:allegro_hand_right sequence="3" parent="base_link" x="-0.2" covers="0" palm="0" phalanges="0" tips="default"/> -->
+	<!-- <xacro:allegro_hand_right sequence="2" parent="world" x="0.2" tips="curved" /> -->
+	<!-- <xacro:allegro_hand_right sequence="3" parent="world" x="-0.2" covers="0" palm="0" phalanges="0" tips="default"/> -->
 </robot>
