Commit message: 'Update 2110041600'

File: xela_models/urdf/xela.xacro (robot description, xacro)
@@ -3,5 +3,5 @@
   <!-- Rviz colors -->
   <material name="black">
-    <color rgba="0.0 0.0 0.0 1.0"/>
+    <color rgba="0.1 0.1 0.1 1.0"/>
   </material>
   <material name="blue">
@@ -408,5 +408,11 @@
   <!-- Allegro Hands -->
   <xacro:macro name="allegro_hand_right" params="sequence parent x:=0.0 y:=0.0 z:=0.0 rx:=0.0 ry:=0.0 rz:=0.0 covers:=1 phalanges:=1 tips:='flat' palm:=1 taxels:=0 defaultnames:=0">
-    <link name="${sequence}_base_link">
+    <xacro:if value="${sequence == ''}">
+      <xacro:property name="seq" value=""/>
+    </xacro:if>
+    <xacro:unless value="${sequence == ''}">
+      <xacro:property name="seq" value="${sequence}_"/>
+    </xacro:unless>
+    <link name="${seq}base_link">
       <visual>
         <geometry>
@@ -444,18 +450,18 @@
       </xacro:if>
     </link>
-    <joint name="${sequence}_ahr_fixed" type="fixed">
+    <joint name="${seq}ahr_fixed" type="fixed">
         <origin xyz="${x} ${y} ${z}" rpy="${radians(rx)} ${radians(ry)} ${radians(rz)}"/>
         <parent link="${parent}" />
-        <child link="${sequence}_base_link" />
+        <child link="${seq}base_link" />
       </joint>
     <xacro:if value="${palm == 1}">
-      <xacro:sensor4x6 sequence="${sequence}_ahr_palm_1" col="red" parent="${sequence}_base_link" x="0.013" y="-0.051" z="-0.0365"  rz="90" rx="90" ry="0.0" taxels="${taxels}" skipinertia="1" />
-      <xacro:sensor4x6 sequence="${sequence}_ahr_palm_2" col="green" parent="${sequence}_base_link" x="0.013" y="0.0523" z="-0.005"  rz="90" rx="90" ry="180.0" taxels="${taxels}" skipinertia="1" />
-      <xacro:sensor4x6 sequence="${sequence}_ahr_palm_3" col="blue" parent="${sequence}_base_link" x="0.013" y="-0.051" z="-0.068" rz="90" rx="90" ry="0.0" taxels="${taxels}" skipinertia="1" />
+      <xacro:sensor4x6 sequence="${seq}ahr_palm_1" col="red" parent="${seq}base_link" x="0.013" y="-0.051" z="-0.0365"  rz="90" rx="90" ry="0.0" taxels="${taxels}" skipinertia="1" />
+      <xacro:sensor4x6 sequence="${seq}ahr_palm_2" col="green" parent="${seq}base_link" x="0.013" y="0.0523" z="-0.005"  rz="90" rx="90" ry="180.0" taxels="${taxels}" skipinertia="1" />
+      <xacro:sensor4x6 sequence="${seq}ahr_palm_3" col="blue" parent="${seq}base_link" x="0.013" y="-0.051" z="-0.068" rz="90" rx="90" ry="0.0" taxels="${taxels}" skipinertia="1" />
     </xacro:if>
     <xacro:if value="${defaultnames == 1}">
     <xacro:finger
-      sequence=			    "${sequence}"
-      parent=				    "${sequence}_base_link"
+      sequence=			    "${seq}"
+      parent=				    "${seq}base_link"
       finger_num=			  "0"
       offset_origin_x=	"${0}"
@@ -469,6 +475,6 @@
     />
     <xacro:finger
-      sequence=			    "${sequence}"
-      parent=				    "${sequence}_base_link"
+      sequence=			    "${seq}"
+      parent=				    "${seq}base_link"
       finger_num=			  "1"
       offset_origin_x=	"${0}"
@@ -482,6 +488,6 @@
     />
     <xacro:finger
-      sequence=			    "${sequence}"
-      parent=				    "${sequence}_base_link"
+      sequence=			    "${seq}"
+      parent=				    "${seq}base_link"
       finger_num=			  "2"
       offset_origin_x=	"${0}"
@@ -495,6 +501,6 @@
     />
     <xacro:thumb_right
-      sequence=			    "${sequence}"
-      parent=				    "${sequence}_base_link"
+      sequence=			    "${seq}"
+      parent=				    "${seq}base_link"
       finger_num=			  "3"
       offset_origin_x=	"-0.0182"
@@ -512,6 +518,6 @@
     <xacro:unless value="${defaultnames == 1}">
       <xacro:finger
-        sequence=			    "${sequence}_hitosashi_finger"
-        parent=				    "${sequence}_base_link"
+        sequence=			    "${seq}hitosashi_finger"
+        parent=				    "${seq}base_link"
         finger_num=			  "0"
         offset_origin_x=	"${0}"
@@ -525,6 +531,6 @@
       />
       <xacro:finger
-        sequence=			    "${sequence}_naka_finger"
-        parent=				    "${sequence}_base_link"
+        sequence=			    "${seq}naka_finger"
+        parent=				    "${seq}base_link"
         finger_num=			  "1"
         offset_origin_x=	"${0}"
@@ -538,6 +544,6 @@
       />
       <xacro:finger
-        sequence=			    "${sequence}_kusuri_finger"
-        parent=				    "${sequence}_base_link"
+        sequence=			    "${seq}kusuri_finger"
+        parent=				    "${seq}base_link"
         finger_num=			  "2"
         offset_origin_x=	"${0}"
@@ -551,6 +557,6 @@
       />
       <xacro:thumb_right
-        sequence=			    "${sequence}_oya_finger"
-        parent=				    "${sequence}_base_link"
+        sequence=			    "${seq}oya_finger"
+        parent=				    "${seq}base_link"
         finger_num=			  "3"
         offset_origin_x=	"-0.0182"

Commit message: 'Update 2110141540'

File: xela_models/urdf/ahrcpcpn.urdf (robot description, URDF)
Before this commit: robot allegro_hand_right, 44 links, 43 joints
Links:
- removed link ahr_palm_1_4x6_base_link
- removed link ahr_palm_2_4x6_base_link
- removed link ahr_palm_3_4x6_base_link
- removed link base_link
- removed link hitosashi_finger_finger_0_aftc_base_link
- removed link hitosashi_finger_finger_link_0
- removed link hitosashi_finger_finger_link_1
- removed link hitosashi_finger_finger_link_1A_4x4_base_link
- removed link hitosashi_finger_finger_link_1B_4x4_base_link
- removed link hitosashi_finger_finger_link_1_cover
- removed link hitosashi_finger_finger_link_2
- removed link hitosashi_finger_finger_link_2_4x4_base_link
- removed link hitosashi_finger_finger_link_2_cover
- removed link hitosashi_finger_finger_link_3
- removed link kusuri_finger_finger_2_aftc_base_link
- removed link kusuri_finger_finger_link_10
- removed link kusuri_finger_finger_link_10_4x4_base_link
- removed link kusuri_finger_finger_link_10_cover
- removed link kusuri_finger_finger_link_11
- removed link kusuri_finger_finger_link_8
- removed link kusuri_finger_finger_link_9
- removed link kusuri_finger_finger_link_9A_4x4_base_link
- removed link kusuri_finger_finger_link_9B_4x4_base_link
- removed link kusuri_finger_finger_link_9_cover
- removed link naka_finger_finger_1_aftc_base_link
- removed link naka_finger_finger_link_4
- removed link naka_finger_finger_link_5
- removed link naka_finger_finger_link_5A_4x4_base_link
- removed link naka_finger_finger_link_5B_4x4_base_link
- removed link naka_finger_finger_link_5_cover
- removed link naka_finger_finger_link_6
- removed link naka_finger_finger_link_6_4x4_base_link
- removed link naka_finger_finger_link_6_cover
- removed link naka_finger_finger_link_7
- removed link oya_finger_3_aftc_base_link
- removed link oya_finger_link_12
- removed link oya_finger_link_13
- removed link oya_finger_link_14
- removed link oya_finger_link_14_4x4_base_link
- removed link oya_finger_link_14_cover
- removed link oya_finger_link_15
- removed link oya_finger_link_15_4x4_base_link
- removed link oya_finger_link_15_cover
- added link 0aftc_palm_link; collision mesh filename=package://xela_models/mesh/ft_c.stl; visual mesh filename=package://xela_models/mesh/ft_c.stl
- added link 1aftc_palm_link; collision mesh filename=package://xela_models/mesh/ft_c.stl; visual mesh filename=package://xela_models/mesh/ft_c.stl
- added link 2aftc_palm_link; collision mesh filename=package://xela_models/mesh/ft_c.stl; visual mesh filename=package://xela_models/mesh/ft_c.stl
- added link 3aftc_palm_link; collision mesh filename=package://xela_models/mesh/ft_c.stl; visual mesh filename=package://xela_models/mesh/ft_c.stl
- added link ahr_palm_1_4x6_palm_link; collision mesh filename=package://xela_models/mesh/4x6.stl; visual mesh filename=package://xela_models/mesh/4x6.stl
- added link ahr_palm_2_4x6_palm_link; collision mesh filename=package://xela_models/mesh/4x6.stl; visual mesh filename=package://xela_models/mesh/4x6.stl
- added link ahr_palm_3_4x6_palm_link; collision mesh filename=package://xela_models/mesh/4x6.stl; visual mesh filename=package://xela_models/mesh/4x6.stl
- added link link_0, mass 0.0127; collision box size=0.0196 0.0275 0.0164; visual mesh filename=package://xela_models/mesh/allegro/link_0.0_ext.STL
- added link link_1, mass 0.0809; collision box size=0.0196 0.0275 0.0164; visual mesh filename=package://xela_models/mesh/allegro/link_1.0.stl
- added link link_10, mass 0.0447; collision box size=0.0196 0.0275 0.054; visual mesh filename=package://xela_models/mesh/allegro/link_2.0.stl
- added link link_10_4x4_palm_link; collision mesh filename=package://xela_models/mesh/4x4.stl; visual mesh filename=package://xela_models/mesh/4x4.stl
- added link link_10_cover; collision mesh filename=package://xela_models/mesh/allegro/link_2_cover.stl; visual mesh filename=package://xela_models/mesh/allegro/link_2_cover.stl
- added link link_11, mass 0.0404; collision box size=0.0196 0.0275 0.026399999999999996; visual mesh filename=package://xela_models/mesh/allegro/link_3.0.STL
- added link link_12, mass 0.0176; collision box size=0.0358 0.034 0.0455; visual mesh filename=package://xela_models/mesh/allegro/link_12.0_right.STL
- added link link_13, mass 0.0127; collision box size=0.0196 0.0275 0.0177; visual mesh filename=package://xela_models/mesh/allegro/link_0.0_ext.STL
- added link link_14, mass 0.0457; collision box size=0.0196 0.0275 0.0514; visual mesh filename=package://xela_models/mesh/allegro/thumb_1.0.stl
- added link link_14_4x4_palm_link; collision mesh filename=package://xela_models/mesh/4x4.stl; visual mesh filename=package://xela_models/mesh/4x4.stl
- added link link_14_cover; collision mesh filename=package://xela_models/mesh/allegro/thumb_1_cover.stl; visual mesh filename=package://xela_models/mesh/allegro/thumb_1_cover.stl
- added link link_15, mass 0.0753; collision box size=0.0196 0.0275 0.042300000000000004; visual mesh filename=package://xela_models/mesh/allegro/thumb_2.0.stl
- added link link_15_4x4_palm_link; collision mesh filename=package://xela_models/mesh/4x4.stl; visual mesh filename=package://xela_models/mesh/4x4.stl
- added link link_15_cover; collision mesh filename=package://xela_models/mesh/allegro/thumb_2_cover.stl; visual mesh filename=package://xela_models/mesh/allegro/thumb_2_cover.stl
- added link link_1A_4x4_palm_link; collision mesh filename=package://xela_models/mesh/4x4.stl; visual mesh filename=package://xela_models/mesh/4x4.stl
- added link link_1B_4x4_palm_link; collision mesh filename=package://xela_models/mesh/4x4.stl; visual mesh filename=package://xela_models/mesh/4x4.stl
- added link link_1_cover; collision mesh filename=package://xela_models/mesh/allegro/link_1_cover.stl; visual mesh filename=package://xela_models/mesh/allegro/link_1_cover.stl
- added link link_2, mass 0.0447; collision box size=0.0196 0.0275 0.054; visual mesh filename=package://xela_models/mesh/allegro/link_2.0.stl
- added link link_2_4x4_palm_link; collision mesh filename=package://xela_models/mesh/4x4.stl; visual mesh filename=package://xela_models/mesh/4x4.stl
- added link link_2_cover; collision mesh filename=package://xela_models/mesh/allegro/link_2_cover.stl; visual mesh filename=package://xela_models/mesh/allegro/link_2_cover.stl
- added link link_3, mass 0.0404; collision box size=0.0196 0.0275 0.026399999999999996; visual mesh filename=package://xela_models/mesh/allegro/link_3.0.STL
- added link link_4, mass 0.0127; collision box size=0.0196 0.0275 0.0164; visual mesh filename=package://xela_models/mesh/allegro/link_0.0_ext.STL
- added link link_5, mass 0.0809; collision box size=0.0196 0.0275 0.0164; visual mesh filename=package://xela_models/mesh/allegro/link_1.0.stl
- added link link_5A_4x4_palm_link; collision mesh filename=package://xela_models/mesh/4x4.stl; visual mesh filename=package://xela_models/mesh/4x4.stl
- added link link_5B_4x4_palm_link; collision mesh filename=package://xela_models/mesh/4x4.stl; visual mesh filename=package://xela_models/mesh/4x4.stl
- added link link_5_cover; collision mesh filename=package://xela_models/mesh/allegro/link_1_cover.stl; visual mesh filename=package://xela_models/mesh/allegro/link_1_cover.stl
- added link link_6, mass 0.0447; collision box size=0.0196 0.0275 0.054; visual mesh filename=package://xela_models/mesh/allegro/link_2.0.stl
- added link link_6_4x4_palm_link; collision mesh filename=package://xela_models/mesh/4x4.stl; visual mesh filename=package://xela_models/mesh/4x4.stl
- added link link_6_cover; collision mesh filename=package://xela_models/mesh/allegro/link_2_cover.stl; visual mesh filename=package://xela_models/mesh/allegro/link_2_cover.stl
- added link link_7, mass 0.0404; collision box size=0.0196 0.0275 0.026399999999999996; visual mesh filename=package://xela_models/mesh/allegro/link_3.0.STL
- added link link_8, mass 0.0127; collision box size=0.0196 0.0275 0.0164; visual mesh filename=package://xela_models/mesh/allegro/link_0.0_ext.STL
- added link link_9, mass 0.0809; collision box size=0.0196 0.0275 0.0164; visual mesh filename=package://xela_models/mesh/allegro/link_1.0.stl
- added link link_9A_4x4_palm_link; collision mesh filename=package://xela_models/mesh/4x4.stl; visual mesh filename=package://xela_models/mesh/4x4.stl
- added link link_9B_4x4_palm_link; collision mesh filename=package://xela_models/mesh/4x4.stl; visual mesh filename=package://xela_models/mesh/4x4.stl
- added link link_9_cover; collision mesh filename=package://xela_models/mesh/allegro/link_1_cover.stl; visual mesh filename=package://xela_models/mesh/allegro/link_1_cover.stl
- added link palm_link, mass 0.4288; collision box size=0.0408 0.1130 0.095; visual mesh filename=package://xela_models/mesh/allegro/base.stl
Joints:
- removed joint hitosashi_finger_finger_0_aftc_fixed
- removed joint hitosashi_finger_finger_joint_0
- removed joint hitosashi_finger_finger_joint_1
- removed joint hitosashi_finger_finger_joint_2
- removed joint hitosashi_finger_finger_joint_3
- removed joint hitosashi_finger_finger_link_1A_4x4_fixed
- removed joint hitosashi_finger_finger_link_1B_4x4_fixed
- removed joint hitosashi_finger_finger_link_1_cover_joint
- removed joint hitosashi_finger_finger_link_2_4x4_fixed
- removed joint hitosashi_finger_finger_link_2_cover_joint
- removed joint kusuri_finger_finger_2_aftc_fixed
- removed joint kusuri_finger_finger_joint_10
- removed joint kusuri_finger_finger_joint_11
- removed joint kusuri_finger_finger_joint_8
- removed joint kusuri_finger_finger_joint_9
- removed joint kusuri_finger_finger_link_10_4x4_fixed
- removed joint kusuri_finger_finger_link_10_cover_joint
- removed joint kusuri_finger_finger_link_9A_4x4_fixed
- removed joint kusuri_finger_finger_link_9B_4x4_fixed
- removed joint kusuri_finger_finger_link_9_cover_joint
- removed joint naka_finger_finger_1_aftc_fixed
- removed joint naka_finger_finger_joint_4
- removed joint naka_finger_finger_joint_5
- removed joint naka_finger_finger_joint_6
- removed joint naka_finger_finger_joint_7
- removed joint naka_finger_finger_link_5A_4x4_fixed
- removed joint naka_finger_finger_link_5B_4x4_fixed
- removed joint naka_finger_finger_link_5_cover_joint
- removed joint naka_finger_finger_link_6_4x4_fixed
- removed joint naka_finger_finger_link_6_cover_joint
- removed joint oya_finger_3_aftc_fixed
- removed joint oya_finger_joint_12
- removed joint oya_finger_joint_13
- removed joint oya_finger_joint_14
- removed joint oya_finger_joint_15
- removed joint oya_finger_link_14_4x4_fixed
- removed joint oya_finger_link_14_cover_joint
- removed joint oya_finger_link_15_4x4_fixed
- removed joint oya_finger_link_15_cover_joint
- added joint 0aftc_fixed: type fixed, parent link_3, child 0aftc_palm_link, origin xyz=-0.013 0.0 0.016 rpy=1.5707963267948966 0.0 1.5707963267948966
- added joint 1aftc_fixed: type fixed, parent link_7, child 1aftc_palm_link, origin xyz=-0.013 0.0 0.016 rpy=1.5707963267948966 0.0 1.5707963267948966
- added joint 2aftc_fixed: type fixed, parent link_11, child 2aftc_palm_link, origin xyz=-0.013 0.0 0.016 rpy=1.5707963267948966 0.0 1.5707963267948966
- added joint 3aftc_fixed: type fixed, parent link_15, child 3aftc_palm_link, origin xyz=-0.013 0.0 0.0315 rpy=1.5707963267948966 0.0 1.5707963267948966
- added joint joint_0: type revolute, parent palm_link, child link_0, origin xyz=0 0.0435 -0.001542 rpy=-0.08726646259971647 0 0, axis 0 0 1, limit lower=-0.47 upper=0.47 effort=15 velocity=7
- added joint joint_1: type revolute, parent link_0, child link_1, origin xyz=0 0 0.0189, axis 0 1 0, limit lower=-0.19599999999999998 upper=1.6099999999999999 effort=15 velocity=7
- added joint joint_10: type revolute, parent link_9, child link_10, origin xyz=0 0 0.054, axis 0 1 0, limit lower=-0.17400000000000002 upper=1.7089999999999999 effort=15 velocity=7
- added joint joint_11: type revolute, parent link_10, child link_11, origin xyz=0 0.0 0.0384, axis 0 1 0, limit lower=-0.227 upper=1.6179999999999999 effort=15 velocity=7
- added joint joint_12: type revolute, parent palm_link, child link_12, origin xyz=-0.0182 0.019333 -0.046487 rpy=0 -1.6580627893946132 -1.5707963267948966, axis -1 0 0, limit lower=0.263 upper=1.396 effort=15 velocity=7
- added joint joint_13: type revolute, parent link_12, child link_13, origin xyz=-0.027 0.005 0.0399, axis 0 0 1, limit lower=-0.10499999999999998 upper=1.1629999999999998 effort=15 velocity=7
- added joint joint_14: type revolute, parent link_13, child link_14, origin xyz=0 0 0.019700000000000002 rpy=0 -0.017453292519943295 0, axis 0 1 0, limit lower=-0.18899999999999997 upper=1.644 effort=15 velocity=7
- added joint joint_15: type revolute, parent link_14, child link_15, origin xyz=0 0 0.0514, axis 0 1 0, limit lower=-0.162 upper=1.7189999999999999 effort=15 velocity=7
- added joint joint_2: type revolute, parent link_1, child link_2, origin xyz=0 0 0.054, axis 0 1 0, limit lower=-0.17400000000000002 upper=1.7089999999999999 effort=15 velocity=7
- added joint joint_3: type revolute, parent link_2, child link_3, origin xyz=0 0.0 0.0384, axis 0 1 0, limit lower=-0.227 upper=1.6179999999999999 effort=15 velocity=7
- added joint joint_4: type revolute, parent palm_link, child link_4, origin xyz=0 0 0.0007 rpy=0.0 0 0, axis 0 0 1, limit lower=-0.47 upper=0.47 effort=15 velocity=7
- added joint joint_5: type revolute, parent link_4, child link_5, origin xyz=0 0 0.0189, axis 0 1 0, limit lower=-0.19599999999999998 upper=1.6099999999999999 effort=15 velocity=7
- added joint joint_6: type revolute, parent link_5, child link_6, origin xyz=0 0 0.054, axis 0 1 0, limit lower=-0.17400000000000002 upper=1.7089999999999999 effort=15 velocity=7
- added joint joint_7: type revolute, parent link_6, child link_7, origin xyz=0 0.0 0.0384, axis 0 1 0, limit lower=-0.227 upper=1.6179999999999999 effort=15 velocity=7
- added joint joint_8: type revolute, parent palm_link, child link_8, origin xyz=0 -0.0435 -0.001542 rpy=0.08726646259971647 0 0, axis 0 0 1, limit lower=-0.47 upper=0.47 effort=15 velocity=7
- added joint joint_9: type revolute, parent link_8, child link_9, origin xyz=0 0 0.0189, axis 0 1 0, limit lower=-0.19599999999999998 upper=1.6099999999999999 effort=15 velocity=7
- added joint link_10_4x4_fixed: type fixed, parent link_10, child link_10_4x4_palm_link, origin xyz=0.01 -0.012 0.0445 rpy=0.0 1.5707963267948966 0.0
- added joint link_10_cover_joint: type fixed, parent link_10, child link_10_cover, origin xyz=0.0 0.0 0.0 rpy=0.0 0.0 0.0
- added joint link_14_4x4_fixed: type fixed, parent link_14, child link_14_4x4_palm_link, origin xyz=0.011 -0.012 0.023 rpy=0.0 1.5707963267948966 0.0
- added joint link_14_cover_joint: type fixed, parent link_14, child link_14_cover, origin xyz=0.0 0.0 0.0 rpy=0.0 0.0 0.0
- added joint link_15_4x4_fixed: type fixed, parent link_15, child link_15_4x4_palm_link, origin xyz=0.011 -0.012 0.021 rpy=0.0 1.5707963267948966 0.0
- added joint link_15_cover_joint: type fixed, parent link_15, child link_15_cover, origin xyz=0.0 0.0 0.0 rpy=0.0 0.0 0.0
- added joint link_1A_4x4_fixed: type fixed, parent link_1, child link_1A_4x4_palm_link, origin xyz=0.0108 0.012 0.033 rpy=0.0 -1.5707963267948966 3.141592653589793
- added joint link_1B_4x4_fixed: type fixed, parent link_1, child link_1B_4x4_palm_link, origin xyz=0.0108 -0.012 0.021 rpy=0.0 1.5707963267948966 0.0
- added joint link_1_cover_joint: type fixed, parent link_1, child link_1_cover, origin xyz=0.0 0.0 0.0 rpy=0.0 0.0 0.0
- added joint link_2_4x4_fixed: type fixed, parent link_2, child link_2_4x4_palm_link, origin xyz=0.01 -0.012 0.0445 rpy=0.0 1.5707963267948966 0.0
- added joint link_2_cover_joint: type fixed, parent link_2, child link_2_cover, origin xyz=0.0 0.0 0.0 rpy=0.0 0.0 0.0
- added joint link_5A_4x4_fixed: type fixed, parent link_5, child link_5A_4x4_palm_link, origin xyz=0.0108 0.012 0.033 rpy=0.0 -1.5707963267948966 3.141592653589793
- added joint link_5B_4x4_fixed: type fixed, parent link_5, child link_5B_4x4_palm_link, origin xyz=0.0108 -0.012 0.021 rpy=0.0 1.5707963267948966 0.0
- added joint link_5_cover_joint: type fixed, parent link_5, child link_5_cover, origin xyz=0.0 0.0 0.0 rpy=0.0 0.0 0.0
- added joint link_6_4x4_fixed: type fixed, parent link_6, child link_6_4x4_palm_link, origin xyz=0.01 -0.012 0.0445 rpy=0.0 1.5707963267948966 0.0
- added joint link_6_cover_joint: type fixed, parent link_6, child link_6_cover, origin xyz=0.0 0.0 0.0 rpy=0.0 0.0 0.0
- added joint link_9A_4x4_fixed: type fixed, parent link_9, child link_9A_4x4_palm_link, origin xyz=0.0108 0.012 0.033 rpy=0.0 -1.5707963267948966 3.141592653589793
- added joint link_9B_4x4_fixed: type fixed, parent link_9, child link_9B_4x4_palm_link, origin xyz=0.0108 -0.012 0.021 rpy=0.0 1.5707963267948966 0.0
- added joint link_9_cover_joint: type fixed, parent link_9, child link_9_cover, origin xyz=0.0 0.0 0.0 rpy=0.0 0.0 0.0
- joint ahr_fixed: child base_link -> palm_link
- joint ahr_palm_1_4x6_fixed: child ahr_palm_1_4x6_base_link -> ahr_palm_1_4x6_palm_link; parent base_link -> palm_link
- joint ahr_palm_2_4x6_fixed: child ahr_palm_2_4x6_base_link -> ahr_palm_2_4x6_palm_link; parent base_link -> palm_link
- joint ahr_palm_3_4x6_fixed: child ahr_palm_3_4x6_base_link -> ahr_palm_3_4x6_palm_link; parent base_link -> palm_link
