Commit message: Model cleaned up and update-251202

File: xela_models/urdf/aftdn.xacro (robot description, xacro)
@@ -2,9 +2,9 @@
 <robot name="allegro_fingertip_flat" xmlns:xacro="http://www.ros.org/wiki/xacro">
   <xacro:arg name="base_prefix" default="base_" />
-   <xacro:macro name="aftdn" params="x_seq parent x:=0.0 y:=0.0 z:=0.0 rx:=0.0 ry:=0.0 rz:=0.0 col:='blue' skipinertia:=0 standalone:=0 sensor_collision:=1">
+   <xacro:macro name="aftdn" params="sequence parent x:=0.0 y:=0.0 z:=0.0 rx:=0.0 ry:=0.0 rz:=0.0 col:='blue' skipinertia:=0 standalone:=0 sensor_collision:=1">
     <xacro:if value="${standalone == 1}">
       <xacro:include filename="$(find xela_models)/urdf/materials.xacro" />
     </xacro:if>
-    <xacro:property name="sequence" value="$(arg base_prefix)${x_seq}"/>
+    <!-- <xacro:property name="sequence" value="$(arg base_prefix)${x_seq}"/> -->
     <joint name="${sequence}_aftd_fixed" type="fixed">
       <origin xyz="${x-0.013} ${y} ${z}" rpy="${radians(rx)} ${radians(ry)} ${radians(rz)}"/>

File: xela_models/urdf/aftfn.xacro (robot description, xacro)
@@ -2,5 +2,5 @@
 <robot name="allegro_fingertip_flat" xmlns:xacro="http://www.ros.org/wiki/xacro">
   <xacro:arg name="base_prefix" default="base_" />
-  <xacro:macro name="sensoraftfn" params="x_seq parent x:=0.0 y:=0.0 z:=0.0 rx:=0.0 ry:=0.0 rz:=0.0 col:='blue' taxels:=0 skipinertia:=0 standalone:=0 sensor_collision:=1 ">
+  <xacro:macro name="sensoraftfn" params="sequence parent x:=0.0 y:=0.0 z:=0.0 rx:=0.0 ry:=0.0 rz:=0.0 col:='blue' taxels:=0 skipinertia:=0 standalone:=0 sensor_collision:=1 ">
     <xacro:if value="${standalone == 1}">
       <xacro:include filename="$(find xela_models)/urdf/materials.xacro" />
@@ -8,5 +8,5 @@
       <xacro:include filename="$(find xela_models)/urdf/4x6n.xacro" />
     </xacro:if>
-    <xacro:property name="sequence" value="$(arg base_prefix)${x_seq}"/>
+    <!-- <xacro:property name="sequence" value="$(arg base_prefix)${x_seq}"/> -->
     <joint name="${sequence}_aftf_fixed" type="fixed">
       <origin xyz="${x} ${y} ${z}" rpy="${radians(rx)} ${radians(ry)} ${radians(rz)}"/>
@@ -79,5 +79,5 @@
     </joint>
     <xacro:if value="${taxels==1}">
-      <xacro:sensor4x4n sequence="${x_seq}_aftf" x="-0.0111665" y="-0.0116665" parent="${sequence}_aftf_sensorbase_link" body="0" sensor_collision="${sensor_collision}" />
+      <xacro:sensor4x4n sequence="${sequence}_aftf" x="-0.0111665" y="-0.0116665" parent="${sequence}_aftf_sensorbase_link" body="0" sensor_collision="${sensor_collision}" />
     </xacro:if>
   </xacro:macro>

File: xela_models/urdf/allegro_hand_left_new.xacro (robot description, xacro)
@@ -1,4 +1,5 @@
 <?xml version="1.0"?>
-<robot xmlns:xacro="http://www.ros.org/wiki/xacro" name="allegro_hand_right">
+<robot xmlns:xacro="http://www.ros.org/wiki/xacro" name="allegro_hand_left">
+<!-- <robot xmlns:xacro="http://www.ros.org/wiki/xacro" > -->
   <xacro:include filename="$(find xela_models)/urdf/materials.xacro" />
   <xacro:include filename="$(find xela_models)/urdf/taxel_n.xacro" />
@@ -12,5 +13,5 @@
   <xacro:arg name="base_prefix" default="base_" />
   <!-- Allegro Hands -->
-  <xacro:macro name="allegro_hand_right_new" params="sequence parent x:=0.0 y:=0.0 z:=0.0 rx:=0.0 ry:=0.0 rz:=0.0 covers:=1 phalanges:=1 tips:='flat' palm:=1 taxels:=0 defaultnames:=0">
+  <xacro:macro name="allegro_hand_left_new" params="sequence parent x:=0.0 y:=0.0 z:=0.0 rx:=0.0 ry:=0.0 rz:=0.0 covers:=1 phalanges:=1 tips:='flat' palm:=1 taxels:=1 defaultnames:=0 sensor_collision=0">
     <xacro:if value="${sequence == ''}">
       <xacro:property name="seq" value=""/>
@@ -34,11 +35,12 @@
         <geometry>
           <xacro:if value="${palm == 1}">
-            <!-- <mesh filename="package://xela_models/mesh/allegro/base_right.stl" /> -->
-            <mesh filename="package://xela_models/mesh/allegro/base_new_right.stl" scale="0.001 0.001 0.001" />
+            <!-- <mesh filename="package://xela_models/mesh/allegro/base_left.stl" /> -->
+            <mesh filename="package://xela_models/mesh/allegro/base_new_left.stl" scale="0.001 0.001 0.001" />
           </xacro:if>
           <xacro:if value="${palm != 1}">
-            <mesh filename="package://xela_models/mesh/allegro/base_right_ns.stl"/>
+            <mesh filename="package://xela_models/mesh/allegro/base_left_ns.stl"/>
           </xacro:if>
         </geometry>
+        <!-- <origin rpy="${radians(-90)} 0 0" xyz="0 0 0 "/> -->
         <material name="cyan">
           <color rgba="0.0 1.0 1.0 1"/>
@@ -72,76 +74,80 @@
         <parent link="hand_root" />
         <child link="${bseq}palm_link" />
-      </joint>
+    </joint>
     <xacro:if value="${palm == 1}">
-      <!-- <xacro:sensor4x6b sequence="${seq}16" col="red" parent="${bseq}palm_link" x="0.013" y="-0.051" z="-0.0365"  rz="90" rx="90" ry="0.0" taxels="${taxels}" skipinertia="1" /> -->
-      <xacro:uspa46_2409 sequence="${seq}16" col="red" parent="${bseq}palm_link" x="0.014" y="-0.021" z="-0.0204"  rz="90" rx="90" ry="180" taxels="${taxels}" skipinertia="1" />
-      <!-- <xacro:sensor4x6b sequence="${seq}17" col="green" parent="${bseq}palm_link" x="0.013" y="0.0523" z="-0.005"  rz="90" rx="90" ry="180.0" taxels="${taxels}" skipinertia="1" /> -->
-      <xacro:uspa46_2409 sequence="${seq}17" col="green" parent="${bseq}palm_link" x="0.014" y="0.021" z="-0.0204"  rz="90" rx="90" ry="0" taxels="${taxels}" skipinertia="1" />
-      <!-- <xacro:sensor4x6b sequence="${seq}18" col="blue" parent="${bseq}palm_link" x="0.013" y="-0.051" z="-0.068" rz="90" rx="90" ry="0.0" taxels="${taxels}" skipinertia="1" /> -->
-      <xacro:uspa46_2409 sequence="${seq}18" col="blue" parent="${bseq}palm_link" x="0.014" y="-0.021" z="-0.0515" rz="90" rx="90" ry="180" taxels="${taxels}" skipinertia="1" />
+      <!-- <xacro:sensor4x6b sequence="${seq}16" col="red" parent="${bseq}palm_link" x="0.013" y="0.051" z="-0.005"  rz="90" rx="90" ry="180" taxels="${taxels}" skipinertia="1"/> -->
+      <xacro:uspa46_2409 sequence="${seq}16" col="red" parent="${bseq}palm_link" x="0.014" y="0.0249" z="-0.0204"  rz="90" rx="90" ry="180" taxels="${taxels}" skipinertia="1" sensor_collision="${sensor_collision}" />
+      <!-- <xacro:sensor4x6b sequence="${seq}17" col="green" parent="${bseq}palm_link" x="0.013" y="-0.0523" z="-0.0365"  rz="90" rx="90" ry="0" taxels="${taxels}" skipinertia="1" /> -->
+      <xacro:uspa46_2409 sequence="${seq}17" col="green" parent="${bseq}palm_link" x="0.014" y="-0.0249" z="-0.0204"  rz="90" rx="90" ry="0" taxels="${taxels}" skipinertia="1" sensor_collision="${sensor_collision}" />
+      <!-- <xacro:sensor4x6b sequence="${seq}18" col="blue" parent="${bseq}palm_link" x="0.013" y="0.051" z="-0.0367" rz="90" rx="90" ry="180" taxels="${taxels}" skipinertia="1" /> -->
+      <xacro:uspa46_2409 sequence="${seq}18" col="blue" parent="${bseq}palm_link" x="0.014" y="0.0249" z="-0.0515" rz="90" rx="90" ry="180" taxels="${taxels}" skipinertia="1" sensor_collision="${sensor_collision}" />
     </xacro:if>
     <xacro:if value="${defaultnames == 1}">
-		<!-- Index Finger -->
-	  <xacro:finger
-		x_seq=			"${seq}"
-    b_seq=      "${bseq}"
-		parent=				"${bseq}palm_link"
-		finger_num=			"0"
-		offset_origin_x=	"${0}"
-		offset_origin_y=	"${0.0435}"
-		offset_origin_z=	"${-0.001542}"
-		finger_angle_r=		"-${radians(5.0)}"
-		covers=				"${covers}"
-		phalanges=			"${phalanges}"
-		tip=				"${tips}"
-		taxels=				"${taxels}"
-	  />
-		<!-- Middle Finger -->
-	  <xacro:finger
-		x_seq=			"${seq}"
-    b_seq=      "${bseq}"
-		parent=				"${bseq}palm_link"
-		finger_num=			"1"
-		offset_origin_x=	"${0}"
-		offset_origin_y=	"0"
-		offset_origin_z=	"${0.0007}"
-		finger_angle_r=		"0.0"
-		covers=				"${covers}"
-		phalanges=			"${phalanges}"
-		tip=				"${tips}"
-		taxels=				"${taxels}"
-	  />
-		<!-- Ring Finger -->
-	  <xacro:finger
-		x_seq=			"${seq}"
-    b_seq=      "${bseq}"
-		parent=				"${bseq}palm_link"
-		finger_num=			"2"
-		offset_origin_x=	"${0}"
-		offset_origin_y=	"-${0.0435}"
-		offset_origin_z=	"${-0.001542}"
-		finger_angle_r=		"${radians(5.0)}"
-		covers=				"${covers}"
-		phalanges=			"${phalanges}"
-		tip=				"${tips}"
-		taxels=				"${taxels}"
-	  />
-		<!-- Thumb -->
-	  <xacro:thumb_right
-		x_seq=			"${seq}"
-    b_seq=      "${bseq}"
-		parent=				"${bseq}palm_link"
-		finger_num=			"3"
-		offset_origin_x=	"-0.0182"
-		offset_origin_y=	"0.019333"
-		offset_origin_z=	"-0.045987"
-		covers=				"${covers}"
-		finger_angle_r=		"0"
-		finger_angle_p=		"-${radians(95)}"
-		finger_angle_y=		"-${radians(90)}"
-		phalanges=			"${phalanges}"
-		tip=				"${tips}"
-		taxels=				"${taxels}"
-	  />
+      <!-- Index Finger -->
+      <xacro:finger
+        x_seq=			"${seq}"
+        b_seq=      "${bseq}"
+        parent=				"${bseq}palm_link"
+        finger_num=			"0"
+        offset_origin_x=	"${0}"
+        offset_origin_y=	"-${0.0435}"
+        offset_origin_z=	"${-0.001542}"
+        finger_angle_r=		"${radians(5.0)}"
+        covers=				"${covers}"
+        phalanges=			"${phalanges}"
+        tip=				"${tips}"
+        taxels=				"${taxels}"
+        sensor_collision="${sensor_collision}"
+      />
+      <!-- Middle Finger -->
+      <xacro:finger
+      x_seq=			"${seq}"
+      b_seq=      "${bseq}"
+      parent=				"${bseq}palm_link"
+      finger_num=			"1"
+      offset_origin_x=	"${0}"
+      offset_origin_y=	"0"
+      offset_origin_z=	"${0.0007}"
+      finger_angle_r=		"0.0"
+      covers=				"${covers}"
+      phalanges=			"${phalanges}"
+      tip=				"${tips}"
+      taxels=				"${taxels}"
+      sensor_collision="${sensor_collision}"
+      />
+      <!-- Ring Finger -->
+      <xacro:finger
+      x_seq=			"${seq}"
+      b_seq=      "${bseq}"
+      parent=				"${bseq}palm_link"
+      finger_num=			"2"
+      offset_origin_x=	"${0}"
+      offset_origin_y=	"${0.0435}"
+      offset_origin_z=	"${-0.001542}"
+      finger_angle_r=		"-${radians(5.0)}"
+      covers=				"${covers}"
+      phalanges=			"${phalanges}"
+      tip=				"${tips}"
+      taxels=				"${taxels}"
+      sensor_collision="${sensor_collision}"
+      />
+      <!-- Thumb -->
+      <xacro:thumb_left
+      x_seq=			"${seq}"
+      b_seq=      "${bseq}"
+      parent=				"${bseq}palm_link"
+      finger_num=			"3"
+      offset_origin_x=	"-0.0182"
+      offset_origin_y=	"-0.019333"
+      offset_origin_z=	"-0.045987"
+      covers=				"${covers}"
+      finger_angle_r=		"0"
+      finger_angle_p=		"-${radians(95)}"
+      finger_angle_y=		"${radians(90)}"
+      phalanges=			"${phalanges}"
+      tip=				"${tips}"
+      taxels=				"${taxels}"
+      sensor_collision="${sensor_collision}"
+      />
     </xacro:if>
     <xacro:unless value="${defaultnames == 1}">
@@ -159,4 +165,5 @@
         tip=				"${tips}"
         taxels=				"${taxels}"
+        sensor_collision="${sensor_collision}"
       />
       <xacro:finger
@@ -173,4 +180,5 @@
         tip=				"${tips}"
         taxels=				"${taxels}"
+        sensor_collision="${sensor_collision}"
       />
       <xacro:finger
@@ -187,6 +195,7 @@
         tip=				"${tips}"
         taxels=				"${taxels}"
+        sensor_collision="${sensor_collision}"
       />
-      <xacro:thumb_right
+      <xacro:thumb_left
         x_seq=			"${seq}oya_finger_"
         b_seq=      "${bseq}"
@@ -203,9 +212,10 @@
         tip=				"${tips}"
         taxels=				"${taxels}"
+        sensor_collision="${sensor_collision}"
       />
     </xacro:unless>
   </xacro:macro>
    <!--FINGER MACRO-->
-  <xacro:macro name="finger" params="x_seq b_seq parent finger_num offset_origin_x offset_origin_y offset_origin_z finger_angle_r covers:=1 tip:='flat' phalanges:=1 taxels:=0">
+  <xacro:macro name="finger" params="x_seq b_seq parent finger_num offset_origin_x offset_origin_y offset_origin_z finger_angle_r covers:=1 tip:='flat' phalanges:=1 taxels:=0 sensor_collision:=1">
     <!-- <xacro:property name="sequence" value="$(arg base_prefix)"/> -->
     <xacro:property name="sequence" value="${b_seq}"/>
@@ -304,6 +314,6 @@
       </xacro:if>
       <xacro:if value="${phalanges == 1}">
-        <xacro:sensor4x4n x_seq="${x_seq}${finger_num*4+1}" col="red" parent="${sequence}link_${finger_num*4+1}" ry="-90" rz="180" z="0.033" y="0.012" x="0.0108" body="1" taxels="${taxels}" skipinertia="1" />
-        <xacro:sensor4x4n x_seq="${x_seq}${finger_num*4+0}" col="red" parent="${sequence}link_${finger_num*4+1}" ry="90" z="0.021" y="-0.012" x="0.0108" body="1" taxels="${taxels}" skipinertia="1" />
+        <xacro:sensor4x4n sequence="${x_seq}${finger_num*4+1}" col="red" parent="${sequence}link_${finger_num*4+1}" ry="-90" rz="180" z="0.033" y="0.012" x="0.0108" body="1" taxels="${taxels}" skipinertia="1" sensor_collision="${sensor_collision}" />
+        <xacro:sensor4x4n sequence="${x_seq}${finger_num*4+0}" col="red" parent="${sequence}link_${finger_num*4+1}" ry="90" z="0.021" y="-0.012" x="0.0108" body="1" taxels="${taxels}" skipinertia="1" sensor_collision="${sensor_collision}" />
       </xacro:if>
       <joint name="joint_${finger_num*4+1}.0" type="revolute">
@@ -379,5 +389,5 @@
       </xacro:if>
       <xacro:if value="${phalanges == 1}">
-        <xacro:sensor4x4n x_seq="${x_seq}${finger_num*4+2}" col="red" parent="${sequence}link_${finger_num*4+2}" ry="90" z="0.0445" y="-0.012" x="0.01" body="1" taxels="${taxels}" skipinertia="1" />
+        <xacro:sensor4x4n sequence="${x_seq}${finger_num*4+2}" col="red" parent="${sequence}link_${finger_num*4+2}" ry="90" z="0.0445" y="-0.012" x="0.01" body="1" taxels="${taxels}" skipinertia="1" sensor_collision="${sensor_collision}" />
       </xacro:if>
       <joint name="joint_${finger_num*4+2}.0" type="revolute">
@@ -431,15 +441,15 @@
       </joint>
     <xacro:if value="${tip == 'flat'}">
-      <xacro:sensoraftfn x_seq="${x_seq}${finger_num*4+3}" col="red" parent="${sequence}link_${finger_num*4+3}" rx="90" rz="90" z="0.016" taxels="${taxels}" skipinertia="1"/>
+      <xacro:sensoraftfn sequence="${x_seq}${finger_num*4+3}" col="red" parent="${sequence}link_${finger_num*4+3}" rx="90" rz="90" z="0.016" taxels="${taxels}" skipinertia="1"/>
     </xacro:if>
     <xacro:if value="${tip == 'curved'}">
-      <xacro:sensoraftcn x_seq="${x_seq}${finger_num*4+3}" col="red" parent="${sequence}link_${finger_num*4+3}" rx="90" rz="90" z="0.016" taxels="${taxels}" skipinertia="1"/>
+      <xacro:sensoraftcn sequence="${x_seq}${finger_num*4+3}" col="red" parent="${sequence}link_${finger_num*4+3}" rx="90" rz="90" z="0.016" taxels="${taxels}" skipinertia="1" sensor_collision="${sensor_collision}" />
     </xacro:if>
     <xacro:if value="${tip == 'default'}">
-      <xacro:aftdn x_seq="${x_seq}${finger_num*4+3}" col="white" parent="${sequence}link_${finger_num*4+3}" rx="0" rz="0" z="0.027" x="0.013" skipinertia="1"/>
+      <xacro:aftdn sequence="${x_seq}${finger_num*4+3}" col="white" parent="${sequence}link_${finger_num*4+3}" rx="0" rz="0" z="0.027" x="0.013" skipinertia="1"/>
     </xacro:if>
     </xacro:macro>
     <!--THUMB MACRO-->
-    <xacro:macro name="thumb_right" params="x_seq b_seq parent finger_num offset_origin_x offset_origin_y offset_origin_z finger_angle_r finger_angle_p finger_angle_y covers:=1 phalanges:=1 tip:='flat' taxels:=0">
+    <xacro:macro name="thumb_left" params="x_seq b_seq parent finger_num offset_origin_x offset_origin_y offset_origin_z finger_angle_r finger_angle_p finger_angle_y covers:=1 phalanges:=1 tip:='flat' taxels:=0 sensor_collision:=1">
       <!-- <xacro:property name="sequence" value="$(arg base_prefix)"/> -->
       <xacro:property name="sequence" value="${b_seq}"/>
@@ -447,7 +457,8 @@
         <visual>
           <geometry>
-            <mesh filename="package://xela_models/mesh/allegro/link_12.0_right.STL" />
+            <mesh filename="package://xela_models/mesh/allegro/link_12.0_left.STL" />
           </geometry>
           <material name="grey" />
+          <origin rpy="${radians(180)} 0 0" xyz="0 0 0"/>
         </visual>
         <collision>
@@ -455,5 +466,5 @@
             <box size="${0.0358} ${0.0340} ${0.0455}"/>
           </geometry>
-          <origin rpy="0 0 0" xyz="${-0.0358/2+0.0} ${.018/2} ${.029/2}"/>
+          <origin rpy="0 0 0" xyz="${-0.0358/2+0.0} -${.018/2} ${.029/2}"/>
         </collision>
         <inertial>
@@ -464,9 +475,10 @@
       </link>
       <joint name="joint_${finger_num*4+0}.0" type="revolute">
-        <axis xyz="-1 0 0"/>
+        <axis xyz="+1 0 0"/>
         <limit effort="15" velocity="7" lower="${0.363-0.1}" upper="${1.496-0.1}" />
         <parent link="${parent}"/>
         <child link="${sequence}link_${finger_num*4+0}"/>
         <origin rpy="${finger_angle_r} ${finger_angle_p} ${finger_angle_y}" xyz="${offset_origin_x} ${offset_origin_y} ${offset_origin_z}"/>
+        <dynamics damping="3" friction="10"/>
       </joint>
       <link name="${sequence}link_${finger_num*4+1}">
@@ -511,9 +523,12 @@
       </xacro:if>
       <joint name="joint_${finger_num*4+1}.0" type="revolute">
-        <axis xyz="0 0 1"/>
+        <!-- <axis xyz="0 0 1"/> -->
+        <axis xyz="0 0 -1"/>
         <limit effort="15" velocity="7" lower="${-0.205+0.1}" upper="${1.263-0.1}" />
+        <!-- <limit effort="15" velocity="7" lower="${-1.263+0.1}" upper="${0.205-0.1}" /> -->
         <parent link="${sequence}link_${finger_num*4+0}"/>
         <child link="${sequence}link_${finger_num*4+1}"/>
-        <origin xyz="-0.027 0.005 0.0399"/>
+        <origin xyz="-0.027 -0.005 0.0399"/>
+        <dynamics damping="3" friction="5"/>
       </joint>
       <link name="${sequence}link_${finger_num*4+2}">
@@ -581,5 +596,5 @@
       </xacro:if>
       <xacro:if value="${phalanges == 1}">
-        <xacro:sensor4x4n x_seq="${x_seq}${finger_num*4+1}" parent="${sequence}link_${finger_num*4+2}" ry="90" z="0.023" y="-0.012" x="0.011" body="1" taxels="${taxels}" skipinertia="1" />
+        <xacro:sensor4x4n sequence="${x_seq}${finger_num*4+1}" parent="${sequence}link_${finger_num*4+2}" ry="90" z="0.023" y="-0.012" x="0.011" body="1" taxels="${taxels}" skipinertia="1" sensor_collision="${sensor_collision}" />
       </xacro:if>
       <joint name="joint_${finger_num*4+2}.0" type="revolute">
@@ -589,4 +604,5 @@
         <child link="${sequence}link_${finger_num*4+2}"/>
         <origin xyz="0 0 ${0.0177}"/>
+        <dynamics damping="3" friction="10"/>
       </joint>
       <link name="${sequence}link_${finger_num*4+3}">
@@ -681,5 +697,5 @@
       </link>
       <xacro:if value="${phalanges == 1}">
-        <xacro:sensor4x4n x_seq="${x_seq}${finger_num*4+2}" parent="${sequence}link_${finger_num*4+3}" ry="90" z="0.021" y="-0.012" x="0.011" body="1" taxels="${taxels}" skipinertia="1" />
+        <xacro:sensor4x4n sequence="${x_seq}${finger_num*4+2}" parent="${sequence}link_${finger_num*4+3}" ry="90" z="0.021" y="-0.012" x="0.011" body="1" taxels="${taxels}" skipinertia="1" sensor_collision="${sensor_collision}" />
       </xacro:if>
     <joint name="joint_${finger_num*4+3}.0" type="revolute">
@@ -689,13 +705,14 @@
       <child link="${sequence}link_${finger_num*4+3}"/>
       <origin xyz="0 0 ${0.0514}"/>
+      <dynamics damping="3" friction="12"/>
     </joint>
     <xacro:if value="${tip == 'flat'}">
-      <xacro:sensoraftfn x_seq="${x_seq}${finger_num*4+3}" col="green" parent="${sequence}link_${finger_num*4+3}" rx="90" rz="90" z="0.0315" taxels="${taxels}" skipinertia="1" />
+      <xacro:sensoraftfn sequence="${x_seq}${finger_num*4+3}" col="green" parent="${sequence}link_${finger_num*4+3}" rx="90" rz="90" z="0.0315" taxels="${taxels}" skipinertia="1" sensor_collision="${sensor_collision}" />
     </xacro:if>
     <xacro:if value="${tip == 'curved'}">
-      <xacro:sensoraftcn x_seq="${x_seq}${finger_num*4+3}" col="green" parent="${sequence}link_${finger_num*4+3}" rx="90" rz="90" z="0.0315" taxels="${taxels}" skipinertia="1" />
+      <xacro:sensoraftcn sequence="${x_seq}${finger_num*4+3}" col="green" parent="${sequence}link_${finger_num*4+3}" rx="90" rz="90" z="0.0315" taxels="${taxels}" skipinertia="1" sensor_collision="${sensor_collision}" />
     </xacro:if>
     <xacro:if value="${tip == 'default'}">
-      <xacro:aftdn x_seq="${x_seq}${finger_num*4+3}" col="white" parent="${sequence}link_${finger_num*4+3}" rx="0" rz="0" z="0.042" x="0.013" skipinertia="1" />
+      <xacro:aftdn sequence="${x_seq}${finger_num*4+3}" col="white" parent="${sequence}link_${finger_num*4+3}" rx="0" rz="0" z="0.042" x="0.013" skipinertia="1" />
     </xacro:if>
   </xacro:macro>

File: xela_models/urdf/allegro_hand_right_curved.xacro (robot description, xacro)
@@ -5,4 +5,4 @@
 	<link name="world" />
 	<xacro:allegro_hand_right_new sequence="0" tips="curved" parent="world"
-								  defaultnames="1" palm="1" taxels="1" />
+								  defaultnames="1" palm="1" taxels="1" sensor_collision="0" />
 </robot>
