Commit message: Add uSPa11, uSPa22 model

File: xela_models/urdf/all_parts_of_individual_module.xacro (robot description, xacro)
@@ -3,6 +3,8 @@
 <xacro:include filename="$(find xela_models)/urdf/materials.xacro" />
 <xacro:include filename="$(find xela_models)/urdf/taxel_n.xacro" />
+<xacro:include filename="$(find xela_models)/urdf/1x1n.xacro" />
+<xacro:include filename="$(find xela_models)/urdf/1x6n.xacro" />
+<xacro:include filename="$(find xela_models)/urdf/2x2n.xacro" />
 <xacro:include filename="$(find xela_models)/urdf/4x4n.xacro" />
-<xacro:include filename="$(find xela_models)/urdf/1x6n.xacro" />
 <xacro:include filename="$(find xela_models)/urdf/4x6n.xacro" />
 <xacro:include filename="$(find xela_models)/urdf/uSPr2F.xacro" />
@@ -32,6 +34,8 @@
   	<xacro:aftdn 		sequence="3" col="red" parent="base_link"  x="0.2" y="0.0" />
   	<xacro:uspref2  	sequence="4" col="red" parent="base_link" taxels="1" x="-0.15" y="0.015" />
-  	<xacro:sensor1x6n 	sequence="5" col="red" parent="base_link" taxels="1" x="0.1" y="0.1" />
-  	<xacro:sensor4x4n 	sequence="6" col="red" parent="base_link" taxels="1" x="0.0" y="0.1" />
-  	<xacro:sensor4x6n	sequence="7" col="red" parent="base_link" taxels="1" x="-0.15" y="0.1" />
+  	<xacro:sensor1x1n 	sequence="5" col="red" parent="base_link" taxels="1" x="0.2" y="0.1" />
+  	<xacro:sensor1x6n 	sequence="6" col="red" parent="base_link" taxels="1" x="0.15" y="0.1" />
+  	<xacro:sensor2x2n 	sequence="7" col="red" parent="base_link" taxels="1" x="0.1" y="0.1" />
+  	<xacro:sensor4x4n 	sequence="8" col="red" parent="base_link" taxels="1" x="0.0" y="0.1" />
+  	<xacro:sensor4x6n	sequence="9" col="red" parent="base_link" taxels="1" x="-0.15" y="0.1" />
 </robot>

File: xela_models/urdf/uSPr2F.xacro (robot description, xacro)
@@ -17,5 +17,5 @@
     <link name="$(arg base_prefix)${sequence}_uspr2f_link">
       <collision>
-        <origin xyz="0 0 0" rpy="0 0 0" />
+        <origin xyz="0 0 0" rpy="0 1.57 1.57" />
         <geometry>
           <mesh filename="package://xela_models/mesh/uspref2.stl" scale="0.001 0.001 0.001"/>
