Commit message: Fixed link prefix name for sensor base: x_taxel -> base_x_taxel

File: xela_models/urdf/2x1n.xacro (robot description, xacro)
@@ -8,10 +8,11 @@
       <xacro:include filename="$(find xela_models)/urdf/taxel_n.xacro" />
     </xacro:if>
-    <joint name="${sequence}_2x1_fixed" type="fixed">
+    <xacro:property name="bseq" value="$(arg base_prefix)${sequence}"/>
+    <joint name="${bseq}_2x1_fixed" type="fixed">
       <origin xyz="${x} ${y} ${z}" rpy="${radians(rx)} ${radians(ry)} ${radians(rz)}"/>
       <parent link="${parent}" />
-      <child link="${sequence}_2x1_link" />
+      <child link="${bseq}_2x1_link" />
     </joint>
-    <link name="${sequence}_2x1_link">
+    <link name="${bseq}_2x1_link">
       <collision>
         <origin xyz="0 0 0" rpy="0 0 0" />
@@ -37,10 +38,10 @@
       </xacro:if>
     </link>
-    <gazebo reference="${sequence}_2x1_link">
+    <gazebo reference="${bseq}_2x1_link">
       <material>Gazebo/Green</material>
     </gazebo>
     <xacro:if value="${taxels == 1}">
-      <xacro:taxel_n sequence="${sequence}_2x1_01"  x="${1*txstep+xoff}" y="${2*tystep+yoff}" z="${zoff}" parent="${sequence}_2x1_link" sensor_collision="${sensor_collision}" />
-      <xacro:taxel_n sequence="${sequence}_2x1_02"  x="${1*txstep+xoff}" y="${1*tystep+yoff}" z="${zoff}" parent="${sequence}_2x1_link" sensor_collision="${sensor_collision}" />
+      <xacro:taxel_n sequence="${sequence}_2x1_01"  x="${1*txstep+xoff}" y="${2*tystep+yoff}" z="${zoff}" parent="${bseq}_2x1_link" sensor_collision="${sensor_collision}" />
+      <xacro:taxel_n sequence="${sequence}_2x1_02"  x="${1*txstep+xoff}" y="${1*tystep+yoff}" z="${zoff}" parent="${bseq}_2x1_link" sensor_collision="${sensor_collision}" />
     </xacro:if>
   </xacro:macro>

File: xela_models/urdf/2x2n.xacro (robot description, xacro)
@@ -8,10 +8,11 @@
       <xacro:include filename="$(find xela_models)/urdf/taxel_n.xacro" />
     </xacro:if>
-    <joint name="${sequence}_2x2_fixed" type="fixed">
+    <xacro:property name="bseq" value="$(arg base_prefix)${sequence}"/>
+    <joint name="${bseq}_2x2_fixed" type="fixed">
       <origin xyz="${x} ${y} ${z}" rpy="${radians(rx)} ${radians(ry)} ${radians(rz)}"/>
       <parent link="${parent}" />
-      <child link="${sequence}_2x2_link" />
+      <child link="${bseq}_2x2_link" />
     </joint>
-    <link name="${sequence}_2x2_link">
+    <link name="${bseq}_2x2_link">
       <collision>
         <origin xyz="0 0 0" rpy="0 0 0" />
@@ -37,12 +38,12 @@
       </xacro:if>
     </link>
-    <gazebo reference="${sequence}_2x2_link">
+    <gazebo reference="${bseq}_2x2_link">
       <material>Gazebo/Green</material>
     </gazebo>
     <xacro:if value="${taxels == 1}">
-      <xacro:taxel_n sequence="${sequence}_2x2_01"  x="${1*txstep+xoff}" y="${2*tystep+yoff}" z="${zoff}" parent="${sequence}_2x2_link" sensor_collision="${sensor_collision}" />
-      <xacro:taxel_n sequence="${sequence}_2x2_02"  x="${2*txstep+xoff}" y="${2*tystep+yoff}" z="${zoff}" parent="${sequence}_2x2_link" sensor_collision="${sensor_collision}" />
-      <xacro:taxel_n sequence="${sequence}_2x2_03"  x="${1*txstep+xoff}" y="${1*tystep+yoff}" z="${zoff}" parent="${sequence}_2x2_link" sensor_collision="${sensor_collision}" />
-      <xacro:taxel_n sequence="${sequence}_2x2_04"  x="${2*txstep+xoff}" y="${1*tystep+yoff}" z="${zoff}" parent="${sequence}_2x2_link" sensor_collision="${sensor_collision}" />
+      <xacro:taxel_n sequence="${sequence}_2x2_01"  x="${1*txstep+xoff}" y="${2*tystep+yoff}" z="${zoff}" parent="${bseq}_2x2_link" sensor_collision="${sensor_collision}" />
+      <xacro:taxel_n sequence="${sequence}_2x2_02"  x="${2*txstep+xoff}" y="${2*tystep+yoff}" z="${zoff}" parent="${bseq}_2x2_link" sensor_collision="${sensor_collision}" />
+      <xacro:taxel_n sequence="${sequence}_2x2_03"  x="${1*txstep+xoff}" y="${1*tystep+yoff}" z="${zoff}" parent="${bseq}_2x2_link" sensor_collision="${sensor_collision}" />
+      <xacro:taxel_n sequence="${sequence}_2x2_04"  x="${2*txstep+xoff}" y="${1*tystep+yoff}" z="${zoff}" parent="${bseq}_2x2_link" sensor_collision="${sensor_collision}" />
     </xacro:if>
   </xacro:macro>

File: xela_models/urdf/4x4n.xacro (robot description, xacro)
@@ -8,10 +8,11 @@
       <xacro:include filename="$(find xela_models)/urdf/taxel_n.xacro" />
     </xacro:if>
-    <joint name="${sequence}_4x4_fixed" type="fixed">
+    <xacro:property name="bseq" value="$(arg base_prefix)${sequence}"/>
+    <joint name="${bseq}_4x4_fixed" type="fixed">
       <origin xyz="${x} ${y} ${z}" rpy="${radians(rx)} ${radians(ry)} ${radians(rz)}"/>
       <parent link="${parent}" />
-      <child link="${sequence}_4x4_link" />
+      <child link="${bseq}_4x4_link" />
     </joint>
-    <link name="${sequence}_4x4_link">
+    <link name="${bseq}_4x4_link">
       <collision>
         <origin xyz="0 0 0" rpy="0 0 0" />
@@ -37,24 +38,24 @@
       </xacro:if>
     </link>
-    <gazebo reference="${sequence}_4x4_link">
+    <gazebo reference="${bseq}_4x4_link">
       <material>Gazebo/Green</material>
     </gazebo>
     <xacro:if value="${taxels == 1}">
-      <xacro:taxel_n sequence="${sequence}_4x4_01"  x="${1*txstep+xoff}" y="${4*tystep+yoff}" z="${zoff}" parent="${sequence}_4x4_link" sensor_collision="${sensor_collision}" />
-      <xacro:taxel_n sequence="${sequence}_4x4_02"  x="${2*txstep+xoff}" y="${4*tystep+yoff}" z="${zoff}" parent="${sequence}_4x4_link" sensor_collision="${sensor_collision}" />
-      <xacro:taxel_n sequence="${sequence}_4x4_03"  x="${3*txstep+xoff}" y="${4*tystep+yoff}" z="${zoff}" parent="${sequence}_4x4_link" sensor_collision="${sensor_collision}" />
-      <xacro:taxel_n sequence="${sequence}_4x4_04"  x="${4*txstep+xoff}" y="${4*tystep+yoff}" z="${zoff}" parent="${sequence}_4x4_link" sensor_collision="${sensor_collision}" />
-      <xacro:taxel_n sequence="${sequence}_4x4_05"  x="${1*txstep+xoff}" y="${3*tystep+yoff}" z="${zoff}" parent="${sequence}_4x4_link" sensor_collision="${sensor_collision}" />
-      <xacro:taxel_n sequence="${sequence}_4x4_06"  x="${2*txstep+xoff}" y="${3*tystep+yoff}" z="${zoff}" parent="${sequence}_4x4_link" sensor_collision="${sensor_collision}" />
-      <xacro:taxel_n sequence="${sequence}_4x4_07"  x="${3*txstep+xoff}" y="${3*tystep+yoff}" z="${zoff}" parent="${sequence}_4x4_link" sensor_collision="${sensor_collision}" />
-      <xacro:taxel_n sequence="${sequence}_4x4_08"  x="${4*txstep+xoff}" y="${3*tystep+yoff}" z="${zoff}" parent="${sequence}_4x4_link" sensor_collision="${sensor_collision}" />
-      <xacro:taxel_n sequence="${sequence}_4x4_09"  x="${1*txstep+xoff}" y="${2*tystep+yoff}" z="${zoff}" parent="${sequence}_4x4_link" sensor_collision="${sensor_collision}" />
-      <xacro:taxel_n sequence="${sequence}_4x4_10" x="${2*txstep+xoff}" y="${2*tystep+yoff}" z="${zoff}" parent="${sequence}_4x4_link" sensor_collision="${sensor_collision}" />
-      <xacro:taxel_n sequence="${sequence}_4x4_11" x="${3*txstep+xoff}" y="${2*tystep+yoff}" z="${zoff}" parent="${sequence}_4x4_link" sensor_collision="${sensor_collision}" />
-      <xacro:taxel_n sequence="${sequence}_4x4_12" x="${4*txstep+xoff}" y="${2*tystep+yoff}" z="${zoff}" parent="${sequence}_4x4_link" sensor_collision="${sensor_collision}" />
-      <xacro:taxel_n sequence="${sequence}_4x4_13" x="${1*txstep+xoff}" y="${1*tystep+yoff}" z="${zoff}" parent="${sequence}_4x4_link" sensor_collision="${sensor_collision}" />
-      <xacro:taxel_n sequence="${sequence}_4x4_14" x="${2*txstep+xoff}" y="${1*tystep+yoff}" z="${zoff}" parent="${sequence}_4x4_link" sensor_collision="${sensor_collision}" />
-      <xacro:taxel_n sequence="${sequence}_4x4_15" x="${3*txstep+xoff}" y="${1*tystep+yoff}" z="${zoff}" parent="${sequence}_4x4_link" sensor_collision="${sensor_collision}" />
-      <xacro:taxel_n sequence="${sequence}_4x4_16" x="${4*txstep+xoff}" y="${1*tystep+yoff}" z="${zoff}" parent="${sequence}_4x4_link" sensor_collision="${sensor_collision}" />
+      <xacro:taxel_n sequence="${sequence}_4x4_01"  x="${1*txstep+xoff}" y="${4*tystep+yoff}" z="${zoff}" parent="${bseq}_4x4_link" sensor_collision="${sensor_collision}" />
+      <xacro:taxel_n sequence="${sequence}_4x4_02"  x="${2*txstep+xoff}" y="${4*tystep+yoff}" z="${zoff}" parent="${bseq}_4x4_link" sensor_collision="${sensor_collision}" />
+      <xacro:taxel_n sequence="${sequence}_4x4_03"  x="${3*txstep+xoff}" y="${4*tystep+yoff}" z="${zoff}" parent="${bseq}_4x4_link" sensor_collision="${sensor_collision}" />
+      <xacro:taxel_n sequence="${sequence}_4x4_04"  x="${4*txstep+xoff}" y="${4*tystep+yoff}" z="${zoff}" parent="${bseq}_4x4_link" sensor_collision="${sensor_collision}" />
+      <xacro:taxel_n sequence="${sequence}_4x4_05"  x="${1*txstep+xoff}" y="${3*tystep+yoff}" z="${zoff}" parent="${bseq}_4x4_link" sensor_collision="${sensor_collision}" />
+      <xacro:taxel_n sequence="${sequence}_4x4_06"  x="${2*txstep+xoff}" y="${3*tystep+yoff}" z="${zoff}" parent="${bseq}_4x4_link" sensor_collision="${sensor_collision}" />
+      <xacro:taxel_n sequence="${sequence}_4x4_07"  x="${3*txstep+xoff}" y="${3*tystep+yoff}" z="${zoff}" parent="${bseq}_4x4_link" sensor_collision="${sensor_collision}" />
+      <xacro:taxel_n sequence="${sequence}_4x4_08"  x="${4*txstep+xoff}" y="${3*tystep+yoff}" z="${zoff}" parent="${bseq}_4x4_link" sensor_collision="${sensor_collision}" />
+      <xacro:taxel_n sequence="${sequence}_4x4_09"  x="${1*txstep+xoff}" y="${2*tystep+yoff}" z="${zoff}" parent="${bseq}_4x4_link" sensor_collision="${sensor_collision}" />
+      <xacro:taxel_n sequence="${sequence}_4x4_10" x="${2*txstep+xoff}" y="${2*tystep+yoff}" z="${zoff}" parent="${bseq}_4x4_link" sensor_collision="${sensor_collision}" />
+      <xacro:taxel_n sequence="${sequence}_4x4_11" x="${3*txstep+xoff}" y="${2*tystep+yoff}" z="${zoff}" parent="${bseq}_4x4_link" sensor_collision="${sensor_collision}" />
+      <xacro:taxel_n sequence="${sequence}_4x4_12" x="${4*txstep+xoff}" y="${2*tystep+yoff}" z="${zoff}" parent="${bseq}_4x4_link" sensor_collision="${sensor_collision}" />
+      <xacro:taxel_n sequence="${sequence}_4x4_13" x="${1*txstep+xoff}" y="${1*tystep+yoff}" z="${zoff}" parent="${bseq}_4x4_link" sensor_collision="${sensor_collision}" />
+      <xacro:taxel_n sequence="${sequence}_4x4_14" x="${2*txstep+xoff}" y="${1*tystep+yoff}" z="${zoff}" parent="${bseq}_4x4_link" sensor_collision="${sensor_collision}" />
+      <xacro:taxel_n sequence="${sequence}_4x4_15" x="${3*txstep+xoff}" y="${1*tystep+yoff}" z="${zoff}" parent="${bseq}_4x4_link" sensor_collision="${sensor_collision}" />
+      <xacro:taxel_n sequence="${sequence}_4x4_16" x="${4*txstep+xoff}" y="${1*tystep+yoff}" z="${zoff}" parent="${bseq}_4x4_link" sensor_collision="${sensor_collision}" />
     </xacro:if>
   </xacro:macro>

File: xela_models/urdf/4x6n.xacro (robot description, xacro)
@@ -2,4 +2,5 @@
 <robot name="4x6n" xmlns:xacro="http://www.ros.org/wiki/xacro">
   <!-- 4x6 new model -->
+  <xacro:arg name="base_prefix" default="base_" />
   <xacro:macro name="sensor4x6n" params="sequence parent x:=0.0 y:=0.0 z:=0.0 rx:=0.0 ry:=0.0 rz:=0.0 col:='blue' body:=1 taxels:=1 skipinertia:=0 xoff=0.003 yoff=0.002175 zoff=0.005 txstep=0.00724 tystep=0.00717 standalone:=0" >
     <xacro:if value="${standalone == 1}">
@@ -7,10 +8,11 @@
       <xacro:include filename="$(find xela_models)/urdf/taxel_n.xacro" />
     </xacro:if>
-    <joint name="${sequence}_4x6_fixed" type="fixed">
+    <xacro:property name="bseq" value="$(arg base_prefix)${sequence}"/>
+    <joint name="${bseq}_4x6_fixed" type="fixed">
       <origin xyz="${x} ${y} ${z}" rpy="${radians(rx)} ${radians(ry)} ${radians(rz)}"/>
       <parent link="${parent}" />
-      <child link="${sequence}_4x6_link" />
+      <child link="${bseq}_4x6_link" />
     </joint>
-    <link name="${sequence}_4x6_link">
+    <link name="${bseq}_4x6_link">
       <collision>
         <origin xyz="0.026 0.0155 0" rpy="3.14 0 3.14" />
@@ -36,32 +38,32 @@
       </xacro:if>
     </link>
-    <gazebo reference="${sequence}_4x6_link">
+    <gazebo reference="${bseq}_4x6_link">
       <material>Gazebo/Red</material>
     </gazebo>
     <xacro:if value="${taxels == 1}">
-      <xacro:taxel_n sequence="${sequence}_4x6_01" x="${1*txstep+xoff}" y="${4*tystep-yoff}" z="${zoff}" parent="${sequence}_4x6_link" />
-      <xacro:taxel_n sequence="${sequence}_4x6_02" x="${2*txstep+xoff}" y="${4*tystep-yoff}" z="${zoff}" parent="${sequence}_4x6_link" />
-      <xacro:taxel_n sequence="${sequence}_4x6_03" x="${3*txstep+xoff}" y="${4*tystep-yoff}" z="${zoff}" parent="${sequence}_4x6_link" />
-      <xacro:taxel_n sequence="${sequence}_4x6_04" x="${4*txstep+xoff}" y="${4*tystep-yoff}" z="${zoff}" parent="${sequence}_4x6_link" />
-      <xacro:taxel_n sequence="${sequence}_4x6_05" x="${5*txstep+xoff}" y="${4*tystep-yoff}" z="${zoff}" parent="${sequence}_4x6_link" />
-      <xacro:taxel_n sequence="${sequence}_4x6_06" x="${6*txstep+xoff}" y="${4*tystep-yoff}" z="${zoff}" parent="${sequence}_4x6_link" />
-      <xacro:taxel_n sequence="${sequence}_4x6_07" x="${1*txstep+xoff}" y="${3*tystep-yoff}" z="${zoff}" parent="${sequence}_4x6_link" />
-      <xacro:taxel_n sequence="${sequence}_4x6_08" x="${2*txstep+xoff}" y="${3*tystep-yoff}" z="${zoff}" parent="${sequence}_4x6_link" />
-      <xacro:taxel_n sequence="${sequence}_4x6_09" x="${3*txstep+xoff}" y="${3*tystep-yoff}" z="${zoff}" parent="${sequence}_4x6_link" />
-      <xacro:taxel_n sequence="${sequence}_4x6_10" x="${4*txstep+xoff}" y="${3*tystep-yoff}" z="${zoff}" parent="${sequence}_4x6_link" />
-      <xacro:taxel_n sequence="${sequence}_4x6_11" x="${5*txstep+xoff}" y="${3*tystep-yoff}" z="${zoff}" parent="${sequence}_4x6_link" />
-      <xacro:taxel_n sequence="${sequence}_4x6_12" x="${6*txstep+xoff}" y="${3*tystep-yoff}" z="${zoff}" parent="${sequence}_4x6_link" />
-      <xacro:taxel_n sequence="${sequence}_4x6_13" x="${1*txstep+xoff}" y="${2*tystep-yoff}" z="${zoff}" parent="${sequence}_4x6_link" />
-      <xacro:taxel_n sequence="${sequence}_4x6_14" x="${2*txstep+xoff}" y="${2*tystep-yoff}" z="${zoff}" parent="${sequence}_4x6_link" />
-      <xacro:taxel_n sequence="${sequence}_4x6_15" x="${3*txstep+xoff}" y="${2*tystep-yoff}" z="${zoff}" parent="${sequence}_4x6_link" />
-      <xacro:taxel_n sequence="${sequence}_4x6_16" x="${4*txstep+xoff}" y="${2*tystep-yoff}" z="${zoff}" parent="${sequence}_4x6_link" />
-      <xacro:taxel_n sequence="${sequence}_4x6_17" x="${5*txstep+xoff}" y="${2*tystep-yoff}" z="${zoff}" parent="${sequence}_4x6_link" />
-      <xacro:taxel_n sequence="${sequence}_4x6_18" x="${6*txstep+xoff}" y="${2*tystep-yoff}" z="${zoff}" parent="${sequence}_4x6_link" />
-      <xacro:taxel_n sequence="${sequence}_4x6_19" x="${1*txstep+xoff}" y="${1*tystep-yoff}" z="${zoff}" parent="${sequence}_4x6_link" />
-      <xacro:taxel_n sequence="${sequence}_4x6_20" x="${2*txstep+xoff}" y="${1*tystep-yoff}" z="${zoff}" parent="${sequence}_4x6_link" />
-      <xacro:taxel_n sequence="${sequence}_4x6_21" x="${3*txstep+xoff}" y="${1*tystep-yoff}" z="${zoff}" parent="${sequence}_4x6_link" />
-      <xacro:taxel_n sequence="${sequence}_4x6_22" x="${4*txstep+xoff}" y="${1*tystep-yoff}" z="${zoff}" parent="${sequence}_4x6_link" />
-      <xacro:taxel_n sequence="${sequence}_4x6_23" x="${5*txstep+xoff}" y="${1*tystep-yoff}" z="${zoff}" parent="${sequence}_4x6_link" />
-      <xacro:taxel_n sequence="${sequence}_4x6_24" x="${6*txstep+xoff}" y="${1*tystep-yoff}" z="${zoff}" parent="${sequence}_4x6_link" />
+      <xacro:taxel_n sequence="${sequence}_4x6_01" x="${1*txstep+xoff}" y="${4*tystep-yoff}" z="${zoff}" parent="${bseq}_4x6_link" />
+      <xacro:taxel_n sequence="${sequence}_4x6_02" x="${2*txstep+xoff}" y="${4*tystep-yoff}" z="${zoff}" parent="${bseq}_4x6_link" />
+      <xacro:taxel_n sequence="${sequence}_4x6_03" x="${3*txstep+xoff}" y="${4*tystep-yoff}" z="${zoff}" parent="${bseq}_4x6_link" />
+      <xacro:taxel_n sequence="${sequence}_4x6_04" x="${4*txstep+xoff}" y="${4*tystep-yoff}" z="${zoff}" parent="${bseq}_4x6_link" />
+      <xacro:taxel_n sequence="${sequence}_4x6_05" x="${5*txstep+xoff}" y="${4*tystep-yoff}" z="${zoff}" parent="${bseq}_4x6_link" />
+      <xacro:taxel_n sequence="${sequence}_4x6_06" x="${6*txstep+xoff}" y="${4*tystep-yoff}" z="${zoff}" parent="${bseq}_4x6_link" />
+      <xacro:taxel_n sequence="${sequence}_4x6_07" x="${1*txstep+xoff}" y="${3*tystep-yoff}" z="${zoff}" parent="${bseq}_4x6_link" />
+      <xacro:taxel_n sequence="${sequence}_4x6_08" x="${2*txstep+xoff}" y="${3*tystep-yoff}" z="${zoff}" parent="${bseq}_4x6_link" />
+      <xacro:taxel_n sequence="${sequence}_4x6_09" x="${3*txstep+xoff}" y="${3*tystep-yoff}" z="${zoff}" parent="${bseq}_4x6_link" />
+      <xacro:taxel_n sequence="${sequence}_4x6_10" x="${4*txstep+xoff}" y="${3*tystep-yoff}" z="${zoff}" parent="${bseq}_4x6_link" />
+      <xacro:taxel_n sequence="${sequence}_4x6_11" x="${5*txstep+xoff}" y="${3*tystep-yoff}" z="${zoff}" parent="${bseq}_4x6_link" />
+      <xacro:taxel_n sequence="${sequence}_4x6_12" x="${6*txstep+xoff}" y="${3*tystep-yoff}" z="${zoff}" parent="${bseq}_4x6_link" />
+      <xacro:taxel_n sequence="${sequence}_4x6_13" x="${1*txstep+xoff}" y="${2*tystep-yoff}" z="${zoff}" parent="${bseq}_4x6_link" />
+      <xacro:taxel_n sequence="${sequence}_4x6_14" x="${2*txstep+xoff}" y="${2*tystep-yoff}" z="${zoff}" parent="${bseq}_4x6_link" />
+      <xacro:taxel_n sequence="${sequence}_4x6_15" x="${3*txstep+xoff}" y="${2*tystep-yoff}" z="${zoff}" parent="${bseq}_4x6_link" />
+      <xacro:taxel_n sequence="${sequence}_4x6_16" x="${4*txstep+xoff}" y="${2*tystep-yoff}" z="${zoff}" parent="${bseq}_4x6_link" />
+      <xacro:taxel_n sequence="${sequence}_4x6_17" x="${5*txstep+xoff}" y="${2*tystep-yoff}" z="${zoff}" parent="${bseq}_4x6_link" />
+      <xacro:taxel_n sequence="${sequence}_4x6_18" x="${6*txstep+xoff}" y="${2*tystep-yoff}" z="${zoff}" parent="${bseq}_4x6_link" />
+      <xacro:taxel_n sequence="${sequence}_4x6_19" x="${1*txstep+xoff}" y="${1*tystep-yoff}" z="${zoff}" parent="${bseq}_4x6_link" />
+      <xacro:taxel_n sequence="${sequence}_4x6_20" x="${2*txstep+xoff}" y="${1*tystep-yoff}" z="${zoff}" parent="${bseq}_4x6_link" />
+      <xacro:taxel_n sequence="${sequence}_4x6_21" x="${3*txstep+xoff}" y="${1*tystep-yoff}" z="${zoff}" parent="${bseq}_4x6_link" />
+      <xacro:taxel_n sequence="${sequence}_4x6_22" x="${4*txstep+xoff}" y="${1*tystep-yoff}" z="${zoff}" parent="${bseq}_4x6_link" />
+      <xacro:taxel_n sequence="${sequence}_4x6_23" x="${5*txstep+xoff}" y="${1*tystep-yoff}" z="${zoff}" parent="${bseq}_4x6_link" />
+      <xacro:taxel_n sequence="${sequence}_4x6_24" x="${6*txstep+xoff}" y="${1*tystep-yoff}" z="${zoff}" parent="${bseq}_4x6_link" />
     </xacro:if>
   </xacro:macro>
