Commit message: Fixed link prefix name for sensor base: x_taxel -> base_x_taxel

File: xela_models/urdf/aftcn.xacro (robot description, xacro)
@@ -7,10 +7,11 @@
       <xacro:include filename="$(find xela_models)/urdf/taxel_n.xacro" />
     </xacro:if>
-    <joint name="${sequence}_aftc_fixed" type="fixed">
+    <xacro:property name="bseq" value="$(arg base_prefix)${sequence}"/>
+    <joint name="${bseq}_aftc_fixed" type="fixed">
       <origin xyz="${x-0.013} ${y} ${z}" rpy="${radians(rx)} ${radians(ry)} ${radians(rz)}"/>
       <parent link="${parent}" />
-      <child link="${sequence}_aftc_link" />
+      <child link="${bseq}_aftc_link" />
     </joint>
-    <link name="${sequence}_aftc_link">
+    <link name="${bseq}_aftc_link">
       <collision>
         <origin xyz="0 0 0" rpy="0 0 0" />
@@ -35,34 +36,34 @@
     </link>
     <xacro:if value="${taxels == 1}">
-      <xacro:taxel_n sequence="${sequence}_aftc_01" x="0.0101" y="0.0306" z="0.01254" ry="90" rz="30" parent="${sequence}_aftc_link" sensor_collision="${sensor_collision}" />
-      <xacro:taxel_n sequence="${sequence}_aftc_02" x="0.0126" y="0.0236" z="0.01254" ry="90" rz="10" parent="${sequence}_aftc_link" sensor_collision="${sensor_collision}" />
-      <xacro:taxel_n sequence="${sequence}_aftc_03" x="0.0138" y="0.0173" z="0.01254" ry="90" rz="10" parent="${sequence}_aftc_link" sensor_collision="${sensor_collision}" />
-      <xacro:taxel_n sequence="${sequence}_aftc_04" x="0.0143" y="0.0103" z="0.01254" ry="90" parent="${sequence}_aftc_link" sensor_collision="${sensor_collision}" />
-      <xacro:taxel_n sequence="${sequence}_aftc_05" x="0.0143" y="0.0038" z="0.01254" ry="90" parent="${sequence}_aftc_link" sensor_collision="${sensor_collision}" />
-      <xacro:taxel_n sequence="${sequence}_aftc_06" x="0.0098" y="0.0230" z="0.02000" ry="50" rz="10" parent="${sequence}_aftc_link" sensor_collision="${sensor_collision}" />
-      <xacro:taxel_n sequence="${sequence}_aftc_07" x="0.0110" y="0.0167" z="0.02000" ry="50" rz="10" parent="${sequence}_aftc_link" sensor_collision="${sensor_collision}" />
-      <xacro:taxel_n sequence="${sequence}_aftc_08" x="0.0115" y="0.0103" z="0.02000" ry="50" parent="${sequence}_aftc_link" sensor_collision="${sensor_collision}" />
-      <xacro:taxel_n sequence="${sequence}_aftc_09" x="0.0115" y="0.0038" z="0.02000" ry="50" parent="${sequence}_aftc_link" sensor_collision="${sensor_collision}" />
-      <xacro:taxel_n sequence="${sequence}_aftc_10" x="0.0037" y="0.0338" z="0.01730" ry="29" rx="-48" parent="${sequence}_aftc_link" sensor_collision="${sensor_collision}" />
-      <xacro:taxel_n sequence="${sequence}_aftc_11" x="0.0039" y="0.0296" z="0.02155" ry="26" rx="-31" parent="${sequence}_aftc_link" sensor_collision="${sensor_collision}" />
-      <xacro:taxel_n sequence="${sequence}_aftc_12" x="0.0039" y="0.0230" z="0.02444" ry="22" rx="-10" parent="${sequence}_aftc_link" sensor_collision="${sensor_collision}" />
-      <xacro:taxel_n sequence="${sequence}_aftc_13" x="0.0039" y="0.0169" z="0.02544" ry="21" rx="-10" parent="${sequence}_aftc_link" sensor_collision="${sensor_collision}" />
-      <xacro:taxel_n sequence="${sequence}_aftc_14" x="0.0039" y="0.0103" z="0.02574" ry="18" parent="${sequence}_aftc_link" sensor_collision="${sensor_collision}" />
-      <xacro:taxel_n sequence="${sequence}_aftc_15" x="0.0039" y="0.0038" z="0.02574" ry="18" parent="${sequence}_aftc_link" sensor_collision="${sensor_collision}" />
-      <xacro:taxel_n sequence="${sequence}_aftc_16" x="-0.0037" y="0.0338" z="0.01730" ry="-29" rx="-48" parent="${sequence}_aftc_link" sensor_collision="${sensor_collision}" />
-      <xacro:taxel_n sequence="${sequence}_aftc_17" x="-0.0039" y="0.0296" z="0.02155" ry="-26" rx="-31" parent="${sequence}_aftc_link" sensor_collision="${sensor_collision}" />
-      <xacro:taxel_n sequence="${sequence}_aftc_18" x="-0.0039" y="0.0230" z="0.02444" ry="-22" rx="-10" parent="${sequence}_aftc_link" sensor_collision="${sensor_collision}" />
-      <xacro:taxel_n sequence="${sequence}_aftc_19" x="-0.0039" y="0.0169" z="0.02544" ry="-21" rx="-10" parent="${sequence}_aftc_link" sensor_collision="${sensor_collision}" />
-      <xacro:taxel_n sequence="${sequence}_aftc_20" x="-0.0039" y="0.0103" z="0.02574" ry="-18" parent="${sequence}_aftc_link" sensor_collision="${sensor_collision}" />
-      <xacro:taxel_n sequence="${sequence}_aftc_21" x="-0.0039" y="0.0038" z="0.02574" ry="-18" parent="${sequence}_aftc_link" sensor_collision="${sensor_collision}" />
-      <xacro:taxel_n sequence="${sequence}_aftc_22" x="-0.0098" y="0.0230" z="0.02000" ry="-50" rz="-10" parent="${sequence}_aftc_link" sensor_collision="${sensor_collision}" />
-      <xacro:taxel_n sequence="${sequence}_aftc_23" x="-0.0110" y="0.0167" z="0.02000" ry="-50" rz="-10" parent="${sequence}_aftc_link" sensor_collision="${sensor_collision}" />
-      <xacro:taxel_n sequence="${sequence}_aftc_24" x="-0.0115" y="0.0103" z="0.02000" ry="-50" parent="${sequence}_aftc_link" sensor_collision="${sensor_collision}" />
-      <xacro:taxel_n sequence="${sequence}_aftc_25" x="-0.0115" y="0.0038" z="0.02000" ry="-50" parent="${sequence}_aftc_link" sensor_collision="${sensor_collision}" />
-      <xacro:taxel_n sequence="${sequence}_aftc_26" x="-0.0101" y="0.0306" z="0.01254" ry="-90" rz="-30" parent="${sequence}_aftc_link" sensor_collision="${sensor_collision}" />
-      <xacro:taxel_n sequence="${sequence}_aftc_27" x="-0.0126" y="0.0236" z="0.01254" ry="-90" rz="-10" parent="${sequence}_aftc_link" sensor_collision="${sensor_collision}" />
-      <xacro:taxel_n sequence="${sequence}_aftc_28" x="-0.0138" y="0.0173" z="0.01254" ry="-90" rz="-10" parent="${sequence}_aftc_link" sensor_collision="${sensor_collision}" />
-      <xacro:taxel_n sequence="${sequence}_aftc_29" x="-0.0143" y="0.0103" z="0.01254" ry="-90" parent="${sequence}_aftc_link" sensor_collision="${sensor_collision}" />
-      <xacro:taxel_n sequence="${sequence}_aftc_30" x="-0.0143" y="0.0038" z="0.01254" ry="-90" parent="${sequence}_aftc_link" sensor_collision="${sensor_collision}" />
+      <xacro:taxel_n sequence="${sequence}_aftc_01" x="0.0101" y="0.0306" z="0.01254" ry="90" rz="30" parent="${bseq}_aftc_link" sensor_collision="${sensor_collision}" />
+      <xacro:taxel_n sequence="${sequence}_aftc_02" x="0.0126" y="0.0236" z="0.01254" ry="90" rz="10" parent="${bseq}_aftc_link" sensor_collision="${sensor_collision}" />
+      <xacro:taxel_n sequence="${sequence}_aftc_03" x="0.0138" y="0.0173" z="0.01254" ry="90" rz="10" parent="${bseq}_aftc_link" sensor_collision="${sensor_collision}" />
+      <xacro:taxel_n sequence="${sequence}_aftc_04" x="0.0143" y="0.0103" z="0.01254" ry="90" parent="${bseq}_aftc_link" sensor_collision="${sensor_collision}" />
+      <xacro:taxel_n sequence="${sequence}_aftc_05" x="0.0143" y="0.0038" z="0.01254" ry="90" parent="${bseq}_aftc_link" sensor_collision="${sensor_collision}" />
+      <xacro:taxel_n sequence="${sequence}_aftc_06" x="0.0098" y="0.0230" z="0.02000" ry="50" rz="10" parent="${bseq}_aftc_link" sensor_collision="${sensor_collision}" />
+      <xacro:taxel_n sequence="${sequence}_aftc_07" x="0.0110" y="0.0167" z="0.02000" ry="50" rz="10" parent="${bseq}_aftc_link" sensor_collision="${sensor_collision}" />
+      <xacro:taxel_n sequence="${sequence}_aftc_08" x="0.0115" y="0.0103" z="0.02000" ry="50" parent="${bseq}_aftc_link" sensor_collision="${sensor_collision}" />
+      <xacro:taxel_n sequence="${sequence}_aftc_09" x="0.0115" y="0.0038" z="0.02000" ry="50" parent="${bseq}_aftc_link" sensor_collision="${sensor_collision}" />
+      <xacro:taxel_n sequence="${sequence}_aftc_10" x="0.0037" y="0.0338" z="0.01730" ry="29" rx="-48" parent="${bseq}_aftc_link" sensor_collision="${sensor_collision}" />
+      <xacro:taxel_n sequence="${sequence}_aftc_11" x="0.0039" y="0.0296" z="0.02155" ry="26" rx="-31" parent="${bseq}_aftc_link" sensor_collision="${sensor_collision}" />
+      <xacro:taxel_n sequence="${sequence}_aftc_12" x="0.0039" y="0.0230" z="0.02444" ry="22" rx="-10" parent="${bseq}_aftc_link" sensor_collision="${sensor_collision}" />
+      <xacro:taxel_n sequence="${sequence}_aftc_13" x="0.0039" y="0.0169" z="0.02544" ry="21" rx="-10" parent="${bseq}_aftc_link" sensor_collision="${sensor_collision}" />
+      <xacro:taxel_n sequence="${sequence}_aftc_14" x="0.0039" y="0.0103" z="0.02574" ry="18" parent="${bseq}_aftc_link" sensor_collision="${sensor_collision}" />
+      <xacro:taxel_n sequence="${sequence}_aftc_15" x="0.0039" y="0.0038" z="0.02574" ry="18" parent="${bseq}_aftc_link" sensor_collision="${sensor_collision}" />
+      <xacro:taxel_n sequence="${sequence}_aftc_16" x="-0.0037" y="0.0338" z="0.01730" ry="-29" rx="-48" parent="${bseq}_aftc_link" sensor_collision="${sensor_collision}" />
+      <xacro:taxel_n sequence="${sequence}_aftc_17" x="-0.0039" y="0.0296" z="0.02155" ry="-26" rx="-31" parent="${bseq}_aftc_link" sensor_collision="${sensor_collision}" />
+      <xacro:taxel_n sequence="${sequence}_aftc_18" x="-0.0039" y="0.0230" z="0.02444" ry="-22" rx="-10" parent="${bseq}_aftc_link" sensor_collision="${sensor_collision}" />
+      <xacro:taxel_n sequence="${sequence}_aftc_19" x="-0.0039" y="0.0169" z="0.02544" ry="-21" rx="-10" parent="${bseq}_aftc_link" sensor_collision="${sensor_collision}" />
+      <xacro:taxel_n sequence="${sequence}_aftc_20" x="-0.0039" y="0.0103" z="0.02574" ry="-18" parent="${bseq}_aftc_link" sensor_collision="${sensor_collision}" />
+      <xacro:taxel_n sequence="${sequence}_aftc_21" x="-0.0039" y="0.0038" z="0.02574" ry="-18" parent="${bseq}_aftc_link" sensor_collision="${sensor_collision}" />
+      <xacro:taxel_n sequence="${sequence}_aftc_22" x="-0.0098" y="0.0230" z="0.02000" ry="-50" rz="-10" parent="${bseq}_aftc_link" sensor_collision="${sensor_collision}" />
+      <xacro:taxel_n sequence="${sequence}_aftc_23" x="-0.0110" y="0.0167" z="0.02000" ry="-50" rz="-10" parent="${bseq}_aftc_link" sensor_collision="${sensor_collision}" />
+      <xacro:taxel_n sequence="${sequence}_aftc_24" x="-0.0115" y="0.0103" z="0.02000" ry="-50" parent="${bseq}_aftc_link" sensor_collision="${sensor_collision}" />
+      <xacro:taxel_n sequence="${sequence}_aftc_25" x="-0.0115" y="0.0038" z="0.02000" ry="-50" parent="${bseq}_aftc_link" sensor_collision="${sensor_collision}" />
+      <xacro:taxel_n sequence="${sequence}_aftc_26" x="-0.0101" y="0.0306" z="0.01254" ry="-90" rz="-30" parent="${bseq}_aftc_link" sensor_collision="${sensor_collision}" />
+      <xacro:taxel_n sequence="${sequence}_aftc_27" x="-0.0126" y="0.0236" z="0.01254" ry="-90" rz="-10" parent="${bseq}_aftc_link" sensor_collision="${sensor_collision}" />
+      <xacro:taxel_n sequence="${sequence}_aftc_28" x="-0.0138" y="0.0173" z="0.01254" ry="-90" rz="-10" parent="${bseq}_aftc_link" sensor_collision="${sensor_collision}" />
+      <xacro:taxel_n sequence="${sequence}_aftc_29" x="-0.0143" y="0.0103" z="0.01254" ry="-90" parent="${bseq}_aftc_link" sensor_collision="${sensor_collision}" />
+      <xacro:taxel_n sequence="${sequence}_aftc_30" x="-0.0143" y="0.0038" z="0.01254" ry="-90" parent="${bseq}_aftc_link" sensor_collision="${sensor_collision}" />
     </xacro:if>
   </xacro:macro>

File: xela_models/urdf/aftfn.xacro (robot description, xacro)
@@ -8,10 +8,11 @@
       <xacro:include filename="$(find xela_models)/urdf/4x6n.xacro" />
     </xacro:if>
-    <joint name="${sequence}_aftf_fixed" type="fixed">
+    <xacro:property name="bseq" value="$(arg base_prefix)${sequence}"/>
+    <joint name="${bseq}_aftf_fixed" type="fixed">
       <origin xyz="${x} ${y} ${z}" rpy="${radians(rx)} ${radians(ry)} ${radians(rz)}"/>
       <parent link="${parent}" />
-      <child link="${sequence}_aftf_link" />
+      <child link="${bseq}_aftf_link" />
     </joint>
-    <link name="${sequence}_aftf_link">
+    <link name="${bseq}_aftf_link">
       <collision>
         <origin xyz="0 0 0" rpy="0 0 0" />
@@ -35,5 +36,5 @@
       </xacro:if>
     </link>
-    <link name="${sequence}_aftf_sensorbase_link">
+    <link name="${bseq}_aftf_sensorbase_link">
       <visual>
         <geometry>
@@ -49,5 +50,5 @@
       </collision>
     </link>
-    <link name="${sequence}_aftf_sensorbase_pos_link">
+    <link name="${bseq}_aftf_sensorbase_pos_link">
       <visual>
         <geometry>
@@ -63,20 +64,20 @@
       </collision>
     </link>
-    <joint name="${sequence}_aftf_sensor_pos_joint" type="prismatic">
+    <joint name="${bseq}_aftf_sensor_pos_joint" type="prismatic">
       <origin xyz="0.0 0.0140 0.0010" rpy="${radians(-25)} 0.0 0.0"/>
-      <parent link="${sequence}_aftf_link"/>
-      <child link="${sequence}_aftf_sensorbase_pos_link"/>
+      <parent link="${bseq}_aftf_link"/>
+      <child link="${bseq}_aftf_sensorbase_pos_link"/>
       <axis xyz="0 0 1"/>
       <limit effort="100.0" lower="0.000" upper="0.000" velocity="0.5"/>
     </joint>
-    <joint name="${sequence}_aftf_sensor_joint" type="prismatic">
+    <joint name="${bseq}_aftf_sensor_joint" type="prismatic">
       <origin xyz="0.0 0.0 0.0" rpy="0.0 0.0 ${radians(-90)}"/>
-      <parent link="${sequence}_aftf_sensorbase_pos_link"/>
-      <child link="${sequence}_aftf_sensorbase_link"/>
+      <parent link="${bseq}_aftf_sensorbase_pos_link"/>
+      <child link="${bseq}_aftf_sensorbase_link"/>
       <axis xyz="0 0 1"/>
       <limit effort="100.0" lower="0.000" upper="0.000" velocity="0.5"/>
     </joint>
     <xacro:if value="${taxels==1}">
-      <xacro:sensor4x4n sequence="${sequence}_aftf" x="-0.0111665" y="-0.0116665" parent="${sequence}_aftf_sensorbase_link" body="0" sensor_collision="${sensor_collision}" />
+      <xacro:sensor4x4n sequence="${sequence}_aftf" x="-0.0111665" y="-0.0116665" parent="${bseq}_aftf_sensorbase_link" body="0" sensor_collision="${sensor_collision}" />
     </xacro:if>
   </xacro:macro>

File: xela_models/urdf/allegro_hand_left_curved.xacro (robot description, xacro)
@@ -1,7 +1,23 @@
 <?xml version="1.0"?>
 <robot xmlns:xacro="http://www.ros.org/wiki/xacro" name="allegro_hand_left">
+	<!-- Arguments -->
+	<xacro:arg name="taxels" default="1"/>
+	<xacro:arg name="sensor_collision" default="0"/>
+	<xacro:arg name="tips" default="curved"/>
+	<xacro:arg name="sequence" default="0"/>
+	<xacro:arg name="defaultnames" default="1"/>
+	<xacro:arg name="palm" default="1"/>
+	<xacro:arg name="parent" default="world"/>
 	<xacro:include filename="$(find xela_models)/urdf/allegro_hand_left_new.xacro" />
+	<xacro:if value="${xacro.arg('parent') == 'world'}">
 	<link name="world" />
-	<xacro:allegro_hand_left_new sequence="0" tips="curved" parent="world"
-								 defaultnames="1" palm="1" taxels="1" sensor_collision="0" />
+	</xacro:if>
+	<xacro:allegro_hand_left_new
+		sequence="$(arg sequence)"
+		tips="$(arg tips)"
+		parent="$(arg parent)"
+		defaultnames="$(arg defaultnames)"
+		palm="$(arg palm)"
+		taxels="$(arg taxels)"
+		sensor_collision="$(arg sensor_collision)" />
 </robot>

File: xela_models/urdf/allegro_hand_right_curved.xacro (robot description, xacro)
@@ -1,7 +1,23 @@
 <?xml version="1.0"?>
 <robot xmlns:xacro="http://www.ros.org/wiki/xacro" name="allegro_hand_right">
+	<!-- Arguments -->
+	<xacro:arg name="taxels" default="1"/>
+	<xacro:arg name="sensor_collision" default="0"/>
+	<xacro:arg name="tips" default="curved"/>
+	<xacro:arg name="sequence" default="0"/>
+	<xacro:arg name="defaultnames" default="1"/>
+	<xacro:arg name="palm" default="1"/>
+	<xacro:arg name="parent" default="world"/>
 	<xacro:include filename="$(find xela_models)/urdf/allegro_hand_right_new.xacro" />
+	<xacro:if value="${xacro.arg('parent') == 'world'}">
 	<link name="world" />
-	<xacro:allegro_hand_right_new sequence="0" tips="curved" parent="world"
-								  defaultnames="1" palm="1" taxels="1" sensor_collision="0" />
+	</xacro:if>
+	<xacro:allegro_hand_right_new
+		sequence="$(arg sequence)"
+		tips="$(arg tips)"
+		parent="$(arg parent)"
+		defaultnames="$(arg defaultnames)"
+		palm="$(arg palm)"
+		taxels="$(arg taxels)"
+		sensor_collision="$(arg sensor_collision)" />
 </robot>
